File: BoatPi.kicad_sch (KiCad schematic)
At the start: 39 parts, among them J1 1432431, J2 1436987, J3 USB3_A_Stacked, J4 JAE_SIM_Card_SF72S006, J5 MDT420M01002, J6 G45A19071083HR, J7 1436987, J8 1432431, U1 SIM7600E-H, U2 PC817, U3 PC817, U4 PC817, U5 PC817, U6 PC817, U7 PC817, U8 PC817, U9 PC817

Commit message: Test Change
Connections:
- net at Module1.84 (+3.3v_(Output)), R11.1, R13.1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: now also A1.36 (3V3), U1.38 (VBAT), U1.39 (VBAT), U1.62 (VBAT), U1.63 (VBAT)
Changed lines of the file:
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@@
+	)
+	(junction
+		(at 39.37 274.32)
+		(diameter 0)
+		(color 0 0 0 0)
 	)
 	(junction
@@
 	)
 	(junction
+		(at 219.71 132.08)
+		(diameter 0)
+		(color 0 0 0 0)
+	)
+	(junction
 		(at 19.05 368.3)
 		(diameter 0)
@@
 	(wire
 		(pts
+			(xy 39.37 274.32) (xy 39.37 156.21)
+		)
+		(stroke
+			(width 0)
+			(type default)
+		)
+	)
+	(wire
+		(pts
 			(xy 217.17 330.2) (xy 217.17 331.47)
 		)
@@
 	(wire
 		(pts
+			(xy 39.37 156.21) (xy 185.42 156.21)
+		)
+		(stroke
+			(width 0)
+			(type default)
+		)
+	)
+	(wire
+		(pts
 			(xy 76.2 119.38) (xy 151.13 119.38)
 		)
@@
 	(wire
 		(pts
+			(xy 219.71 132.08) (xy 354.33 132.08)
+		)
+		(stroke
+			(width 0)
+			(type default)
+		)
+	)
+	(wire
+		(pts
 			(xy 177.8 372.11) (xy 177.8 328.93)
 		)
@@
 	(wire
 		(pts
+			(xy 185.42 132.08) (xy 219.71 132.08)
+		)
+		(stroke
+			(width 0)
+			(type default)
+		)
+	)
+	(wire
+		(pts
 			(xy 24.13 401.32) (xy 39.37 401.32)
 		)
@@
 	(wire
 		(pts
+			(xy 185.42 156.21) (xy 185.42 132.08)
+		)
+		(stroke
+			(width 0)
+			(type default)
+		)
+	)
+	(wire
+		(pts
 			(xy 77.47 354.33) (xy 58.42 354.33)
 		)
@@
 	(wire
 		(pts
+			(xy 354.33 172.72) (xy 354.33 132.08)
+		)
+		(stroke
+			(width 0)
+			(type default)
+		)
+	)
+	(wire
+		(pts
 			(xy 146.05 223.52) (xy 134.62 223.52)
 		)
@@
 		)
 		(stroke
+			(width 0)
+			(type default)
+		)
+	)
+	(wire
+		(pts
+			(xy 219.71 132.08) (xy 219.71 142.24)
+		)
+		(stroke

Commit message: New Test
Connections:
- net at A1.40 (VBUS): now also Module1.1 (GND)
Changed lines of the file:
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@@
+	(wire
+		(pts
+			(xy 158.75 137.16) (xy 214.63 137.16)
+		)
+		(stroke
+			(width 0)
+			(type default)
+		)
+	)
 	(wire
 		(pts
@@
 	(wire
 		(pts
+			(xy 158.75 170.18) (xy 158.75 137.16)
+		)
+		(stroke
+			(width 0)
+			(type default)
+		)
+	)
+	(wire
+		(pts
 			(xy 55.88 200.66) (xy 55.88 332.74)
 		)
@@
 	(wire
 		(pts
+			(xy 214.63 137.16) (xy 214.63 142.24)
+		)
+		(stroke
+			(width 0)
+			(type default)
+		)
+	)
+	(wire
+		(pts
 			(xy 120.65 392.43) (xy 139.7 392.43)
 		)
@@
 		)
 		(stroke
+			(width 0)
+			(type default)
+		)
+	)
+	(wire
+		(pts
+			(xy 134.62 170.18) (xy 158.75 170.18)
+		)
+		(stroke

Commit message: started PCB
Parts:
- removed J3: USB3_A_Stacked, symbol Connector:USB3_A_Stacked
- removed J5: MDT420M01002, NVMEPretty:AMPHENOL_MDT420M01002, symbol NVME:MDT420M01002
- removed J6: G45A19071083HR, HDMIPretty:AMPHENOL_G45A19071083HR, symbol HDMI:G45A19071083HR
- added C1: EEEFN1J100L, 10uFCapPretty:CAP_EEEFN1J100L, symbol 10uFCap:EEEFN1J100L
- added C2, C6: C1812W104KDRACTU, 100nFCapPretty:CAPC4532X185N, symbol 100nFCap:C1812W104KDRACTU
- added C3, C4: EEEFN1C220R, 22uFCap:CAP_EEEFN1C220R, symbol 22uFCap:EEEFN1C220R
- added C5: JMK316BBJ227ML-TE, 470uFCeramPretty:CAPC3216X190N, symbol 470uFCeram:JMK316BBJ227ML-TE
- added C7, C8: C2012X5R1V106M125AC, 10uFCeramPretty:CAPC2012X145N, symbol 10uFCeram:C2012X5R1V106M125AC
- added J10, J11, J12: CONSMA002-SMD-G, SMAconPretty:TE_CONSMA002-SMD-G, symbol SMAcon:CONSMA002-SMD-G
- added J14: Barrel_Jack_MountingPin, Connector_BarrelJack:BarrelJack_CUI_PJ-063AH_Horizontal, symbol Connector:Barrel_Jack_MountingPin
- added L1, L2: L, Inductor_SMD:L_0805_2012Metric, symbol Device:L
- added R18, R19: R, Resistor_SMD:R_0805_2012Metric, symbol Device:R
- added R20: 7500, Resistor_SMD:R_0805_2012Metric, symbol Device:R
- added R21: 1020, Resistor_SMD:R_0805_2012Metric, symbol Device:R
- added R22: 100k, Resistor_SMD:R_0805_2012Metric, symbol Device:R
- added U10: AP62301WU-7, APBuckPretty:SOT95P280X100-6N, symbol APBuck:AP62301WU-7
- R1, R10, R11, R12, R13, R14, R15, R16, R17, R2, R3, R4, R5, R6, R7, R8, R9: footprint (none) -> Resistor_SMD:R_0805_2012Metric
Connections:
- net at PS1.10_11 (PGND), PS1.12 (PGND): now also J4.C5 (GND), PS1.18 (AGND), PS1.21 (AGND), U1.1 (GND), U1.10 (GND), U1.14 (GND), U1.2 (GND), U1.37 (GND), U1.40 (GND), U1.41 (GND), U1.43 (GND), U1.5 (GND), U1.57 (GND), U1.58 (GND), U1.60 (GND), U1.61 (GND), U1.64 (GND), U1.65 (GND), U1.77 (GND), U1.78 (GND), U1.80 (GND), U1.81 (GND), C1.2, C3.2, C4.2, C5.2, C7.2, C8.2, J10.2, J10.3, J11.2, J11.3, J12.2, J12.3, J14.2, R19.2, R20.2, U10.1 (GND)
- net GND_Page2: now reaches Module1.43 (GND), PS1.13 (VCC)
- net GND_Page2: now also R22.1
- net at PS1.14_15 (SW), PS1.16 (SW), PS1.19_20 (SW)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: now also L2.1
- net 5V_Page2: now reaches Module1.77 (+5v_(Input)), PS1.1_2 (VOUT), PS1.6_7 (VOUT)
- net 5V_Page2: now also A1.39 (VSYS), PS1.25 (SENSE), U1.11 (USB_VBUS), C5.1, C6.2, R21.1
- net at PS1.24 (SEQ): now also C6.1
- net at PS1.26 (FB): now also R20.1, R21.2
- net at J1.5, PS1.27 (+VIN), PS1.28 (+VIN)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: now also PS1.3 (CTRL/UVLO), C1.1, C7.1, C8.1, J14.1, U10.3 (VIN), U10.5 (EN)
- net at PS1.4 (PG): now also R22.2
- net 3.3v_Page2: now reaches A1.36 (3V3), Module1.84 (+3.3v_(Output)), R11.1, R13.1, R15.1, R2.1, R3.1, R5.1, R7.1, R9.1
- net 3.3v_Page2: no longer U1.38 (VBAT), U1.39 (VBAT), U1.62 (VBAT), U1.63 (VBAT)
- net at Module1.65 (GND), NMEA2000_CanController2.2 (VSS): now also A1.13 (GND), A1.18 (GND), A1.23 (GND), A1.28 (GND), A1.3 (GND), A1.33 (AGND), A1.38 (GND), A1.8 (GND); no longer Fuel_ADS1115.3 (GND)
- net at R8.1: no longer U5.1
- net at R8.2: no longer J2.1
- net at A1.40 (VBUS): no longer Module1.1 (GND)
- net at A1.6 (GPIO4): now also Module1.51 (GPIO15)
- net at A1.7 (GPIO5): now also Module1.55 (GPIO14)
- net at J1.4, J8.1: now also Fuel_ADS1115.3 (GND)
- net at J4.C1 (VCC): now also U1.20 (USIM_VDD)
- net at J4.C2 (RST): now also U1.18 (USIM_RST)
- net at J4.C3 (CLK): now also U1.19 (USIM_CLK)
- net at J4.C6 (VPP/SWP): now also U1.17 (USIM_DATA)
- net at Module1.25 (GPIO21): now also U1.3 (PWRKEY)
- net at Module1.27 (GPIO20): now also U1.4 (RESET)
- net PI5_USB3_1_DN: now reaches U1.12 (USB_DN)
- net PI5_USB3_1_DP: now reaches U1.13 (USB_DP)
- net at U1.59 (AUX_ANT): now also J12.1
- net at U1.79 (GNSS_ANT): now also J10.1
- net at U1.82 (MAIN_ANT): now also J11.1
- new net: R18.2, R19.1, U10.4 (FB)
- new net: C3.1, C4.1, L1.1, R18.1, U1.38 (VBAT), U1.39 (VBAT), U1.62 (VBAT), U1.63 (VBAT)
- new net: C2.2, L1.2, U10.2 (SW)
- new net: A1.1 (GPIO0), R7.2, U5.4
- new net: C2.1, U10.6 (BST)
- now unconnected: Module1.10 (Ethernet_Pair0_N), Module1.12 (Ethernet_Pair0_P), Module1.14 (GND), Module1.16 (FAN_TACHO), Module1.18 (Ethernet_SYNC_OUT(3.3v)), Module1.2 (GND), Module1.20 (EEPROM_nWP), Module1.4 (Ethernet_Pair1_P), Module1.6 (Ethernet_Pair1_N), Module1.8 (GND)
- no-connect marks 0 -> 189
Other:
- added sheet Sheet2 (untitled.kicad_sch)
- company: (none) -> RiceElectronics
- title: (none) -> Yamaha Boat Dash
- moved on the sheet: J4, R11, R2, R3, R8

Commit message: At home update
Connections:
- net 3.3v_Page2 is gone; now on net +3.3V: A1.36 (3V3), Module1.84 (+3.3v_(Output)), R11.1, R13.1, R15.1, R2.1, R3.1, R5.1, R7.1, R9.1
- net GND_Page2 is gone; now on net GND: Module1.43 (GND), PS1.13 (VCC), R22.1
- net GND: now reaches C1.2, C3.2, C4.2, J10.2, J10.3, J11.2, J11.3, J12.2, J12.3, J4.C5 (GND), R19.2, U1.1 (GND), U1.10 (GND), U1.14 (GND), U1.2 (GND), U1.37 (GND), U1.40 (GND), U1.41 (GND), U1.43 (GND), U1.5 (GND), U1.57 (GND), U1.58 (GND), U1.60 (GND), U1.61 (GND), U1.64 (GND), U1.65 (GND), U1.77 (GND), U1.78 (GND), U1.80 (GND), U1.81 (GND), U10.1 (GND)
- net GND: now also A1.13 (GND), A1.18 (GND), A1.23 (GND), A1.28 (GND), A1.3 (GND), A1.33 (AGND), A1.38 (GND), A1.8 (GND), Module1.98 (GND), NMEA2000_CanController2.2 (VSS), U2.3, U3.3, U4.3, U5.3, U6.3, U7.3, U8.3, U9.3; no longer C5.2, C7.2, C8.2, J14.2, PS1.10_11 (PGND), PS1.12 (PGND), PS1.18 (AGND), PS1.21 (AGND), R20.2
- net +3.3V: now reaches Module1.86 (+3.3v_(Output)), NMEA2000_CanController2.3 (VDD), R17.2
- net +3.3V: no longer Fuel_ADS1115.8 (VDD)
- net 5V_Page2 renamed +5V
- net +5V: no longer U1.11 (USB_VBUS)
- new net: C5.2, C7.2, C8.2, J14.2, PS1.10_11 (PGND), PS1.12 (PGND), PS1.18 (AGND), PS1.21 (AGND), R20.2
- now unconnected: Module1.65 (GND)

Commit message: Updated from work
Parts:
- removed A1: RaspberryPi_Pico_W, Module:RaspberryPi_Pico_W_SMD, symbol MCU_Module:RaspberryPi_Pico_W
- added A1: RaspberryPi_Pico, Module:RaspberryPi_Pico_SMD_HandSolder, symbol MCU_Module:RaspberryPi_Pico
- added M2: Fan_CPU_4pin, Connector:FanPinHeader_1x04_P2.54mm_Vertical, symbol Motor:Fan_CPU_4pin
Connections:
- net +3.3V: now also A1.36 (3V3)
- net +5V: now also A1.39 (VSYS), M2.2 (+)
- net GND: now also A1.13 (GND), A1.18 (GND), A1.23 (GND), A1.28 (GND), A1.3 (GND), A1.33 (AGND), A1.38 (GND), A1.8 (GND), M2.1 (-)
- net at R8.1: now also U5.1
- net at R8.2: now also J2.1
- net at R7.2, U5.4: now also A1.1 (GPIO0)
- net at R9.2, U6.4: now also A1.2 (GPIO1)
- net at NMEA2000_CanController2.1 (TXD): now also A1.27 (GPIO21)
- net at NMEA2000_CanController2.4 (RXD): now also A1.29 (GPIO22)
- net at Module1.51 (GPIO15): now also A1.6 (GPIO4)
- net at Module1.55 (GPIO14): now also A1.7 (GPIO5)
- net at Module1.16 (FAN_TACHO): now also M2.3 (Tacho)
- net at Module1.19 (FAN_PWM): now also M2.4 (PWM)
- no-connect marks 189 -> 187
Other:
- moved on the sheet: R8

Commit message: Fixed scheme
Parts:
- U1: footprint Sim7600Pretty:IC_SIM7600E-H -> SIM7600E-H:IC_SIM7600E-H
- U10: footprint APBuckPretty:SOT95P280X100-6N -> AP62301WU-7:SOT95P280X100-6N
Connections:
- net +3.3V: now also Fuel_ADS1115.8 (VDD); no longer A1.36 (3V3), Module1.86 (+3.3v_(Output))
- net GND: now also Fuel_ADS1115.3 (GND), J1.4, J8.1, Module1.65 (GND), PS1.10_11 (PGND), PS1.12 (PGND), PS1.18 (AGND), PS1.21 (AGND), R20.2; no longer A1.33 (AGND), PS1.13 (VCC), R22.1
- net at C1.1, C7.1, C8.1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: now also Module1.27 (GPIO20), U1.4 (RESET)
- new net: PS1.13 (VCC), R22.1
- new net: C5.2, C7.2, C8.2, J14.2
- no-connect marks 187 -> 190

Commit message: Home push
Parts:
- added C9: 10uf, Capacitor_SMD:C_0805_2012Metric, symbol Device:C
- added J9: Micro_SD_Card_Det2, Connector_Card:SD_TE_2041021, symbol Connector:Micro_SD_Card_Det2
- added R23: 12k, Resistor_SMD:R_0805_2012Metric, symbol Device:R
- added U11: RT9742BGJ5F, Package_TO_SOT_SMD:TSOT-23-5, symbol Power_Management:RT9742BGJ5F
Connections:
- net +3.3V: now also Module1.78 (GPIO_VREF(1.8v/3.3v_Input)), Module1.86 (+3.3v_(Output)), R23.1, U11.5 (VIN)
- net GND: now also C9.2, J9.11 (SHIELD), J9.6 (VSS), U11.2 (GND)
- net at Module1.57 (SD_CLK): now also J9.5 (CLK)
- net at Module1.61 (SD_DAT3): now also J9.2 (DAT3/CD)
- net at Module1.62 (SD_CMD): now also J9.3 (CMD)
- net at Module1.63 (SD_DAT0): now also J9.7 (DAT0)
- net at Module1.67 (SD_DAT1): now also J9.8 (DAT1)
- net at Module1.69 (SD_DAT2): now also J9.1 (DAT2)
- net at Module1.75 (SD_PWR_ON): now also R23.2, U11.4 (~{EN})
- new net: C9.1, J9.4 (VDD), U11.1 (VOUT)
- no-connect marks 190 -> 184

Commit message: Work Changes and documentation
Parts:
- added F1: 3550-2, NewFuseHolderPretty:FUSE_3550-2, symbol NewFuseHolder:3550-2
Connections:
- net +5V: now also U1.11 (USB_VBUS)
- net at C1.1, C7.1, C8.1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: now also F1.2_1, F1.2_2; no longer J14.1
- net PI5_USB3_1_DN renamed USB_DN
- net PI5_USB3_1_DP renamed USB_DP
- new net: F1.1_1, F1.1_2, J14.1
