File: BoatPi.kicad_sch (KiCad schematic)
At the start: 62 parts, among them J1 1432431, J10 CONSMA002-SMD-G, J11 CONSMA002-SMD-G, J12 CONSMA002-SMD-G, J14 Barrel_Jack_MountingPin, J2 1436987, J4 JAE_SIM_Card_SF72S006, J7 1436987, J8 1432431, J9 Micro_SD_Card_Det2, M2 Fan_CPU_4pin, U1 SIM7600E-H, U10 AP62301WU-7, U11 RT9742BGJ5F, U2 PC817, U3 PC817, U4 PC817, U5 PC817, U6 PC817, U7 PC817, U8 PC817, U9 PC817

Commit message: PCIE Changes
Parts:
- removed A1: RaspberryPi_Pico, Module:RaspberryPi_Pico_SMD_HandSolder, symbol MCU_Module:RaspberryPi_Pico
- added J6: 1436987, PHPretty:1436987, symbol PH168873061:1436987
- added K1: Relay_SPDT, Relay_THT:Relay_SPDT_Finder_36.11, symbol Relay:Relay_SPDT
- added U16: SC0917, Pico2Pretty:MODULE_SC0917, symbol Pico2:SC0917
- U1: footprint SIM7600E-H:IC_SIM7600E-H -> Sim7600Pretty:IC_SIM7600E-H
- U10: footprint AP62301WU-7:SOT95P280X100-6N -> APBuckPretty:SOT95P280X100-6N
Connections:
- net +3.3V: now also J6.3
- net +5V: now also U16.39 (VSYS)
- net GND: now also C5.2, C7.2, C8.2, J14.2, Module1.1 (GND), Module1.13 (GND), Module1.14 (GND), Module1.2 (GND), Module1.22 (GND), Module1.23 (GND), Module1.32 (GND), Module1.33 (GND), Module1.42 (GND), Module1.52 (GND), Module1.53 (GND), Module1.59 (GND), Module1.60 (GND), Module1.66 (GND), Module1.7 (GND), Module1.71 (GND), Module1.74 (GND), Module1.8 (GND), J6.4, J6.5, K1.A2, U16.13 (GND), U16.18 (GND), U16.23 (GND), U16.28 (GND), U16.3 (GND), U16.33 (AGND), U16.38 (GND), U16.8 (GND), U16.A (USB_SHIELD), U16.B (USB_SHIELD), U16.C (USB_SHIELD), U16.D (USB_SHIELD), U16.D2 (GND)
- net at R7.2, U5.4: now also U16.1 (GP0)
- net at R9.2, U6.4: now also U16.2 (GP1)
- net at NMEA2000_CanController2.1 (TXD): now also U16.27 (GP21)
- net at NMEA2000_CanController2.4 (RXD): now also U16.29 (GP22)
- net at Module1.51 (GPIO15): now also U16.11 (GP8)
- net at Module1.55 (GPIO14): now also U16.12 (GP9)
- net at C1.1, C7.1, C8.1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: now also K1.14; no longer F1.2_1, F1.2_2, Module1.27 (GPIO20), U1.4 (RESET)
- net GPIO8: now reaches Module1.39 (GPIO8)
- net GPIO8: now also J6.8
- net GPIO25: now reaches Module1.41 (GPIO25)
- net GPIO25: now also J6.7
- net GPIO24: now reaches Module1.45 (GPIO24)
- net GPIO24: now also J6.6
- new net: F1.2_1, F1.2_2, J6.1, K1.11
- new net: J6.2, K1.A1
- new net: Module1.27 (GPIO20), U1.4 (RESET)
- no-connect marks 184 -> 169

Commit message: diff pairs
Connections:
- net GND: now also J1.1, J1.5, J1.MH1, NMEA2000_CanController2.8 (STBY); no longer J1.4
- net at C1.1, C7.1, C8.1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: now also J1.4; no longer J1.5
- net CAN-: now reaches J1.2
- net CAN-: now also NMEA2000_CanController2.7 (CANH); no longer NMEA2000_CanController2.8 (STBY)
- net CAN+: now reaches J1.3, NMEA2000_CanController2.6 (CANL)
- no-connect marks 169 -> 166
Changed lines of the file:
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@@
 	)
 	(junction
+		(at 297.18 400.05)
+		(diameter 0)
+		(color 0 0 0 0)
+	)
+	(junction
 		(at 393.7 276.86)
 		(diameter 0)
@@
 	)
 	(no_connect
-		(at 285.75 382.27)
-	)
-	(no_connect
 		(at 308.61 248.92)
 	)
@@
 	)
 	(no_connect
-		(at 297.18 402.59)
-	)
-	(no_connect
 		(at 354.33 210.82)
 	)
@@
 	)
 	(no_connect
-		(at 274.32 397.51)
-	)
-	(no_connect
 		(at 354.33 203.2)
 	)
@@
 	(wire
 		(pts
+			(xy 267.97 402.59) (xy 274.32 402.59)
+		)
+		(stroke
+			(width 0)
+			(type default)
+		)
+	)
+	(wire
+		(pts
 			(xy 44.45 359.41) (xy 44.45 368.3)
 		)
@@
 	(wire
 		(pts
-			(xy 269.24 388.62) (xy 288.29 388.62)
+			(xy 269.24 388.62) (xy 285.75 388.62)
 		)
 		(stroke
@@
 	(wire
 		(pts
-			(xy 459.74 388.62) (xy 459.74 138.43)
+			(xy 459.74 386.08) (xy 459.74 138.43)
 		)
 		(stroke
@@
 	(wire
 		(pts
+			(xy 297.18 397.51) (xy 306.07 397.51)
+		)
+		(stroke
+			(width 0)
+			(type default)
+		)
+	)
+	(wire
+		(pts
 			(xy 100.33 119.38) (xy 100.33 123.19)
 		)
@@
 	(wire
 		(pts
-			(xy 288.29 388.62) (xy 288.29 382.27)
-		)
-		(stroke
-			(width 0)
-			(type default)
-		)
-	)
-	(wire
-		(pts
 			(xy 180.34 292.1) (xy 190.5 292.1)
 		)
@@
 	(wire
 		(pts
-			(xy 297.18 400.05) (xy 306.07 400.05)
-		)
-		(stroke
-			(width 0)
-			(type default)
-		)
-	)
-	(wire
-		(pts
 			(xy 19.05 360.68) (xy 19.05 354.33)
 		)
@@
 	(wire
 		(pts
-			(xy 274.32 402.59) (xy 267.97 402.59)
-		)
-		(stroke
-			(width 0)
-			(type default)
-		)
-	)
-	(wire
-		(pts
 			(xy 309.88 143.51) (xy 316.23 143.51)
 		)
@@
 	(wire
 		(pts
-			(xy 306.07 400.05) (xy 306.07 388.62)
+			(xy 306.07 397.51) (xy 306.07 386.08)
 		)
 		(stroke
@@
 	(wire
 		(pts
+			(xy 285.75 382.27) (xy 285.75 388.62)
+		)
+		(stroke
+			(width 0)
+			(type default)
+		)
+	)
+	(wire
+		(pts
 			(xy 35.56 124.46) (xy 31.75 124.46)
 		)
@@
 	(wire
 		(pts
+			(xy 297.18 400.05) (xy 297.18 402.59)
+		)
+		(stroke
+			(width 0)
+			(type default)
+		)
+	)
+	(wire
+		(pts
 			(xy 100.33 119.38) (xy 119.38 119.38)
 		)
@@
 	(wire
 		(pts
-			(xy 306.07 388.62) (xy 459.74 388.62)
+			(xy 306.07 386.08) (xy 459.74 386.08)
 		)
 		(stroke
@@
 		)
 	)
+	(label "CAN+"
+		(at 269.24 402.59 0)
+		(effects
+			(font
+				(size 1.27 1.27)
+			)
+			(justify left bottom)
+		)
+	)
+	(label "CAN-"
+		(at 270.51 400.05 0)
+		(effects
+			(font
+				(size 1.27 1.27)
+			)
+			(justify left bottom)
+		)
+	)
 	(global_label "GPIO24"
 		(shape input)
@@
 	(symbol
 		(lib_id "power:GND")
+		(at 274.32 397.51 180)
+		(unit 1)
+		(exclude_from_sim no)
+		(in_bom yes)
+		(on_board yes)
+		(dnp no)
+		(fields_autoplaced yes)
+		(property "Reference" "#PWR0105"
+			(at 274.32 391.16 0)
+			(effects
+				(font
+					(size 1.27 1.27)
+				)
+				(hide yes)
+			)
+		)
+		(property "Value" "GND"
+			(at 274.32 392.43 0)
+			(effects
+				(font
+					(size 1.27 1.27)
+				)
+			)
+		)
+		(property "Footprint" ""
+			(at 274.32 397.51 0)
+			(effects
+				(font
+					(size 1.27 1.27)
+				)
+				(hide yes)
+			)
+		)
+		(property "Datasheet" ""
+			(at 274.32 397.51 0)
+			(effects
+				(font
+					(size 1.27 1.27)
+				)
+				(hide yes)
+			)
+		)
+		(property "Description" "Power symbol creates a global label with name \"GND\" , ground"
+			(at 274.32 397.51 0)
+			(effects
+				(font
+					(size 1.27 1.27)
+				)
+				(hide yes)
+			)
+		)
+		(pin "1"
+		)
+		(instances
+			(project "BoatPi"
+				(path "/f5624df3-0379-482b-a515-d4dba6ca8ab3"
+					(reference "#PWR0105")
+					(unit 1)
+				)
+			)
+		)
+	)
+	(symbol
+		(lib_id "power:GND")
 		(at 66.04 293.37 0)
 		(unit 1)
@@
 	(symbol
 		(lib_id "power:GND")
-		(at 297.18 397.51 180)
+		(at 297.18 400.05 90)
 		(unit 1)
 		(exclude_from_sim no)
@@
 		(fields_autoplaced yes)
 		(property "Reference" "#PWR025"
-			(at 297.18 391.16 0)
+			(at 303.53 400.05 0)
 			(effects
 				(font
@@
 		)
 		(property "Value" "GND"
-			(at 297.18 392.43 0)
+			(at 300.99 400.0499 90)
 			(effects
 				(font
 					(size 1.27 1.27)
 				)
+				(justify right)
 			)
 		)
 		(property "Footprint" ""
-			(at 297.18 397.51 0)
+			(at 297.18 400.05 0)
 			(effects
 				(font
@@
 		)
 		(property "Datasheet" ""
-			(at 297.18 397.51 0)
+			(at 297.18 400.05 0)
 			(effects
 				(font
@@
 		)
 		(property "Description" "Power symbol creates a global label with name \"GND\" , ground"
-			(at 297.18 397.51 0)
+			(at 297.18 400.05 0)
 			(effects
 				(font
@@
 					(unit 1)
 				)
+			)
+		)
+	)
+	(symbol
+		(lib_id "power:GND")
+		(at 288.29 382.27 0)
+		(unit 1)
+		(exclude_from_sim no)
+		(in_bom yes)
+		(on_board yes)
+		(dnp no)
+		(fields_autoplaced yes)
+		(property "Reference" "#PWR0104"
+			(at 288.29 388.62 0)
+			(effects
+				(font
+					(size 1.27 1.27)
+				)
+				(hide yes)
+			)
+		)
+		(property "Value" "GND"
+			(at 288.29 387.35 0)
+			(effects
+				(font
+					(size 1.27 1.27)
+				)
+			)
+		)
+		(property "Footprint" ""
+			(at 288.29 382.27 0)
+			(effects
+				(font
+					(size 1.27 1.27)
+				)
+				(hide yes)
+			)
+		)
+		(property "Datasheet" ""
+			(at 288.29 382.27 0)
+			(effects
+				(font
+					(size 1.27 1.27)
+				)
+				(hide yes)
+			)
+		)
+		(property "Description" "Power symbol creates a global label with name \"GND\" , ground"
+			(at 288.29 382.27 0)
+			(effects
+				(font
+					(size 1.27 1.27)
+				)
+				(hide yes)
+			)
+		)
+		(pin "1"
+		)
+		(instances
+			(project ""
+				(path "/f5624df3-0379-482b-a515-d4dba6ca8ab3"
+					(reference "#PWR0104")
+					(unit 1)
+				)

Commit message: Fixes from datasheets
Parts:
- removed C1: EEEFN1J100L, 10uFCapPretty:CAP_EEEFN1J100L, symbol 10uFCap:EEEFN1J100L
- removed C3, C4: EEEFN1C220R, 22uFCap:CAP_EEEFN1C220R, symbol 22uFCap:EEEFN1C220R
- removed L1: L, Inductor_SMD:L_0805_2012Metric, symbol Device:L
- removed U10: AP62301WU-7, APBuckPretty:SOT95P280X100-6N, symbol APBuck:AP62301WU-7
- added C1: C_Polarized_Small_US, Capacitor_SMD:C_0805_2012Metric, symbol Device:C_Polarized_Small_US
- added C25, C29: 100nF, Capacitor_SMD:C_0805_2012Metric, symbol Device:C
- added C26, C27, C28: 22pF_NM, Capacitor_SMD:C_0805_2012Metric, symbol Device:C
- added D2: ESDA6V1W5, TVSPretty:SOT65P210X110-5N, symbol TVS:ESDA6V1W5
- added D3: TVS-bidirectional Diode, Diode_SMD:D_0805_2012Metric, symbol SimTVS:TVS-bidirectional-Diode
- added F2: 2A, Fuse:Fuse_0805_2012Metric, symbol Device:Fuse
- added Q2: BC107, Package_TO_SOT_THT:TO-18-3, symbol Transistor_BJT:BC107
- added R29, R30, R31: 22 Ohm, Resistor_SMD:R_0805_2012Metric, symbol Device:R
- added R32: 0 Ohm, Resistor_SMD:R_0805_2012Metric, symbol Device:R
- added R33: 4.7K, Resistor_SMD:R_0805_2012Metric, symbol Device:R
- added R34: 47k, Resistor_SMD:R_0805_2012Metric, symbol Device:R
- added R35: 470R, Resistor_SMD:R_0805_2012Metric, symbol Device:R
- added U10: MIC29302AWU, Package_TO_SOT_SMD:TO-263-5_TabPin3, symbol Regulator_Linear:MIC29302AWU
- J9: footprint Connector_Card:SD_TE_2041021 -> CM5IO:SDCARD_MOLEX_503398-1892
- R18, R19: value R -> 470R
Connections:
- net +5V: now also F2.1
- net GND: now also C2.2, J4.SH, R18.2, C1.2, C25.1, C26.1, C27.1, C28.1, C29.1, D2.2, D3.1 (K), Q2.1 (E), R32.1, R34.1, U10.3 (GND)
- net at R19.1: now also R35.2, U10.5 (ADJ); no longer R18.2
- net at R18.1, U1.38 (VBAT), U1.39 (VBAT)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: now also C2.1, C1.1, R35.1, U10.4 (VOUT)
- net GPIO3: now reaches Fuel_ADS1115.10 (SCL)
- net GPIO3: now also Module1.56 (GPIO3)
- net GPIO2: now reaches Fuel_ADS1115.9 (SDA)
- net GPIO2: now also Module1.58 (GPIO2)
- net at J4.C1 (VCC), U1.20 (USIM_VDD): now also C25.2, D2.1
- net at J4.C2 (RST), U1.18 (USIM_RST): now also J4.C7 (I/O), C28.2, D2.3, D2.5, R29.2, R31.1, R31.2
- net at U1.19 (USIM_CLK): now also C27.2, R30.1; no longer J4.C3 (CLK)
- net at J4.C6 (VPP/SWP): no longer U1.17 (USIM_DATA)
- net at J4.CSW: now also J4.DSW, U1.53 (USIM_DET)
- net at Module1.25 (GPIO21): no longer U1.3 (PWRKEY)
- net at U1.4 (RESET): now also C29.2, D3.2 (A), Q2.3 (C); no longer Module1.27 (GPIO20)
- new net: Q2.2 (B), R33.1, R34.2
- new net: F2.2, U10.1 (EN), U10.2 (VIN)
- new net: Module1.27 (GPIO20), R33.2
- new net: D2.4, J4.C3 (CLK), R30.2
- new net: C26.2, R29.1, U1.17 (USIM_DATA)
- new net: R32.2, U1.3 (PWRKEY)
- no-connect marks 166 -> 159
Other:
- moved on the sheet: C2, J4

Commit message: Final Updates
Connections:
- net +3.3V: no longer NMEA2000_CanController2.3 (VDD)
- net +5V: now also NMEA2000_CanController2.3 (VDD)
- new net: C28.2, R31.1, U1.18 (USIM_RST)
- new net: D2.3, J4.C2 (RST), R31.2
- new net: D2.5, J4.C7 (I/O), R29.2
Changed lines of the file:
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@@
 	)
 	(junction
+		(at 334.01 311.15)
+		(diameter 0)
+		(color 0 0 0 0)
+	)
+	(junction
 		(at 346.71 303.53)
 		(diameter 0)
@@
 	)
 	(junction
-		(at 344.17 312.42)
-		(diameter 0)
-		(color 0 0 0 0)
-	)
-	(junction
 		(at 82.55 359.41)
 		(diameter 0)
@@
 	)
 	(junction
-		(at 334.01 312.42)
-		(diameter 0)
-		(color 0 0 0 0)
-	)
-	(junction
 		(at 95.25 354.33)
 		(diameter 0)
@@
 	(wire
 		(pts
+			(xy 326.39 280.67) (xy 326.39 285.75)
+		)
+		(stroke
+			(width 0)
+			(type default)
+		)
+	)
+	(wire
+		(pts
 			(xy 378.46 158.75) (xy 370.84 158.75)
 		)
@@
 	(wire
 		(pts
-			(xy 334.01 312.42) (xy 334.01 323.85)
+			(xy 334.01 311.15) (xy 334.01 323.85)
 		)
 		(stroke
@@
 	(wire
 		(pts
-			(xy 373.38 316.23) (xy 373.38 312.42)
+			(xy 373.38 316.23) (xy 373.38 311.15)
 		)
 		(stroke
@@
 	(wire
 		(pts
-			(xy 334.01 308.61) (xy 334.01 312.42)
+			(xy 334.01 308.61) (xy 334.01 311.15)
 		)
 		(stroke
@@
 	(wire
 		(pts
-			(xy 344.17 285.75) (xy 326.39 285.75)
+			(xy 344.17 280.67) (xy 326.39 280.67)
 		)
 		(stroke
@@
 	(wire
 		(pts
-			(xy 344.17 312.42) (xy 334.01 312.42)
-		)
-		(stroke
-			(width 0)
-			(type default)
-		)
-	)
-	(wire
-		(pts
 			(xy 280.67 187.96) (xy 280.67 321.31)
 		)
@@
 	(wire
 		(pts
-			(xy 344.17 285.75) (xy 344.17 312.42)
+			(xy 344.17 280.67) (xy 344.17 312.42)
 		)
 		(stroke
@@
 	(wire
 		(pts
-			(xy 344.17 320.04) (xy 344.17 312.42)
-		)
-		(stroke
-			(width 0)
-			(type default)
-		)
-	)
-	(wire
-		(pts
 			(xy 100.33 130.81) (xy 100.33 133.35)
 		)
@@
 	(wire
 		(pts
-			(xy 373.38 312.42) (xy 344.17 312.42)
+			(xy 334.01 311.15) (xy 373.38 311.15)
 		)
 		(stroke
@@
 	)
 	(symbol
-		(lib_id "power:+3.3V")
-		(at 283.21 316.23 0)
-		(unit 1)
-		(exclude_from_sim no)
-		(in_bom yes)
-		(on_board yes)
-		(dnp no)
-		(fields_autoplaced yes)
-		(property "Reference" "#PWR09"
-			(at 283.21 320.04 0)
-			(effects
-				(font
-					(size 1.27 1.27)
-				)
-				(hide yes)
-			)
-		)
-		(property "Value" "+3.3V"
-			(at 283.21 311.15 0)
-			(effects
-				(font
-					(size 1.27 1.27)
-				)
-			)
-		)
-		(property "Footprint" ""
-			(at 283.21 316.23 0)
-			(effects
-				(font
-					(size 1.27 1.27)
-				)
-				(hide yes)
-			)
-		)
-		(property "Datasheet" ""
-			(at 283.21 316.23 0)
-			(effects
-				(font
-					(size 1.27 1.27)
-				)
-				(hide yes)
-			)
-		)
-		(property "Description" "Power symbol creates a global label with name \"+3.3V\""
-			(at 283.21 316.23 0)
-			(effects
-				(font
-					(size 1.27 1.27)
-				)
-				(hide yes)
-			)
-		)
-		(pin "1"
-		)
-		(instances
-			(project ""
-				(path "/f5624df3-0379-482b-a515-d4dba6ca8ab3"
-					(reference "#PWR09")
-					(unit 1)
-				)
-			)
-		)
-	)
-	(symbol
 		(lib_id "power:GND")
 		(at 361.95 182.88 0)
@@
 		(on_board yes)
 		(dnp no)
-		(fields_autoplaced yes)
 		(property "Reference" "NMEA2000_CanController2"
-			(at 294.64 350.5199 90)
+			(at 294.386 355.6 90)
 			(effects
 				(font
@@
 					(unit 1)
 				)
+			)
+		)
+	)
+	(symbol
+		(lib_id "power:+5V")
+		(at 283.21 316.23 0)
+		(unit 1)
+		(exclude_from_sim no)
+		(in_bom yes)
+		(on_board yes)
+		(dnp no)
+		(fields_autoplaced yes)
+		(property "Reference" "#PWR09"
+			(at 283.21 320.04 0)
+			(effects
+				(font
+					(size 1.27 1.27)
+				)
+				(hide yes)
+			)
+		)
+		(property "Value" "+5V"
+			(at 283.21 311.15 0)
+			(effects
+				(font
+					(size 1.27 1.27)
+				)
+			)
+		)
+		(property "Footprint" ""
+			(at 283.21 316.23 0)
+			(effects
+				(font
+					(size 1.27 1.27)
+				)
+				(hide yes)
+			)
+		)
+		(property "Datasheet" ""
+			(at 283.21 316.23 0)
+			(effects
+				(font
+					(size 1.27 1.27)
+				)
+				(hide yes)
+			)
+		)
+		(property "Description" "Power symbol creates a global label with name \"+5V\""
+			(at 283.21 316.23 0)
+			(effects
+				(font
+					(size 1.27 1.27)
+				)
+				(hide yes)
+			)
+		)
+		(pin "1"
+		)
+		(instances
+			(project ""
+				(path "/f5624df3-0379-482b-a515-d4dba6ca8ab3"
+					(reference "#PWR09")
+					(unit 1)
+				)
