File: BoatPi.kicad_pcb (KiCad board)
At the start: 2 copper layers, 59 parts, among them J1 1432431, J10 CONSMA002-SMD-G, J11 CONSMA002-SMD-G, J12 CONSMA002-SMD-G, J13 HDMI_A_1.4, J14 Barrel_Jack_MountingPin, J2 1436987, J3 Bus_M.2_Socket_M, J4 JAE_SIM_Card_SF72S006, J5 USB3_A, J6 USB3_A, J7 1436987, J8 1432431, U1 SIM7600E-H, U10 AP62301WU-7, U2 PC817, U3 PC817, U4 PC817, U5 PC817, U6 PC817, U7 PC817, U8 PC817, U9 PC817

Commit message: At home update
Parts:
- moved J4 404.7 mm to (547.4, 312.3)
- moved J5 246.2 mm to (413.2, 314.0)
- moved J6 246.2 mm to (440.7, 314.0)
- moved C2 237.0 mm to (586.4, 230.0)
- moved R19 233.6 mm to (593.5, 231.9), turned to 90 degrees
- moved J10 229.3 mm to (567.9, 311.0)
- moved J3 226.6 mm to (407.2, 198.0)
- moved U10 226.4 mm to (574.8, 230.9)
- moved A1 222.9 mm to (296.4, 195.9)
- moved J2 222.9 mm to (282.4, 294.9)
- moved J7 222.9 mm to (329.4, 295.9)
- moved J8 222.9 mm to (491.4, 308.9)
- moved L2 222.9 mm to (261.5, 156.9)
- moved PS1 222.9 mm to (253.7, 159.5)
- moved R1 222.9 mm to (275.4, 279.0)
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Connections:
- A1 pad 13: Net-(A1-AGND) -> GND
- A1 pad 18: Net-(A1-AGND) -> GND
- A1 pad 23: Net-(A1-AGND) -> GND
- A1 pad 28: Net-(A1-AGND) -> GND
- A1 pad 3: Net-(A1-AGND) -> GND
- A1 pad 33: Net-(A1-AGND) -> GND
- A1 pad 36: 3.3v_Page2 -> +3.3V
- A1 pad 38: Net-(A1-AGND) -> GND
- A1 pad 39: /5V_Page2 -> +5V
- A1 pad 8: Net-(A1-AGND) -> GND
- C1 pad 2: Net-(J4-GND) -> GND
- C3 pad 2: Net-(J4-GND) -> GND
- C4 pad 2: Net-(J4-GND) -> GND
- C5 pad 1: /5V_Page2 -> +5V
- C5 pad 2: Net-(J4-GND) -> Net-(C5-Pad2)
- C7 pad 2: Net-(J4-GND) -> Net-(C5-Pad2)
- C8 pad 2: Net-(J4-GND) -> Net-(C5-Pad2)
- Fuel_ADS1115 pad 8: Net-(Fuel_ADS1115-VDD) -> unconnected-(Fuel_ADS1115-VDD-Pad8)
- J10 pad 2: Net-(J4-GND) -> GND
- J10 pad 3: Net-(J4-GND) -> GND
- J11 pad 2: Net-(J4-GND) -> GND
- J11 pad 3: Net-(J4-GND) -> GND
- J12 pad 2: Net-(J4-GND) -> GND
- J12 pad 3: Net-(J4-GND) -> GND
- J13 pad 11: /Sheet2/GND -> GND
- J13 pad 17: /Sheet2/GND -> GND
- J13 pad 18: /Sheet2/+5v -> +5V
- J13 pad 2: /Sheet2/GND -> GND
- J13 pad 5: /Sheet2/GND -> GND
- J13 pad 8: /Sheet2/GND -> GND
- J14 pad 2: Net-(J4-GND) -> Net-(C5-Pad2)
- J3 pad 1: /Sheet2/GND -> GND
- J3 pad 12: /Sheet2/+3.3v -> +3.3V
- J3 pad 14: /Sheet2/+3.3v -> +3.3V
- J3 pad 15: /Sheet2/GND -> GND
- J3 pad 16: /Sheet2/+3.3v -> +3.3V
- J3 pad 18: /Sheet2/+3.3v -> +3.3V
- J3 pad 2: /Sheet2/+3.3v -> +3.3V
- J3 pad 21: /Sheet2/GND -> GND
- J3 pad 27: /Sheet2/GND -> GND
- J3 pad 3: /Sheet2/GND -> GND
- J3 pad 33: /Sheet2/GND -> GND
- J3 pad 39: /Sheet2/GND -> GND
- J3 pad 4: /Sheet2/+3.3v -> +3.3V
- J3 pad 45: /Sheet2/GND -> GND
- J3 pad 51: /Sheet2/GND -> GND
- J3 pad 53: unconnected-(J3-REFCLKn-Pad53) -> Net-(J3-REFCLKn)
- J3 pad 55: unconnected-(J3-REFCLKp-Pad55) -> Net-(J3-REFCLKp)
- J3 pad 57: /Sheet2/GND -> GND
- J3 pad 70: /Sheet2/+3.3v -> +3.3V
- J3 pad 71: /Sheet2/GND -> GND
- J3 pad 72: /Sheet2/+3.3v -> +3.3V
- J3 pad 73: /Sheet2/GND -> GND
- J3 pad 74: /Sheet2/+3.3v -> +3.3V
- J3 pad 75: /Sheet2/GND -> GND
- J3 pad 9: /Sheet2/GND -> GND
- J4 pad C5: Net-(J4-GND) -> GND
- J5 pad 10: Net-(J5-SHIELD) -> GND
- J6 pad 10: Net-(J5-SHIELD) -> GND
- Module1 pad 108: /Sheet2/GND -> GND
- Module1 pad 110: unconnected-(Module1B-PCIe_CLK_P-Pad110) -> Net-(J3-REFCLKp)
- Module1 pad 112: unconnected-(Module1B-PCIe_CLK_N-Pad112) -> Net-(J3-REFCLKn)
- Module1 pad 191: /Sheet2/GND -> GND
- Module1 pad 192: Net-(J5-SHIELD) -> GND
- Module1 pad 43: /GND_Page2 -> GND
- Module1 pad 65: Net-(A1-AGND) -> unconnected-(Module1A-GND-Pad65)
- Module1 pad 77: /5V_Page2 -> +5V
- Module1 pad 84: 3.3v_Page2 -> +3.3V
- Module1 pad 86: Net-(Fuel_ADS1115-VDD) -> +3.3V
- Module1 pad 98: Net-(Module1A-GND-Pad98) -> GND
- NMEA2000_CanController2 pad 2: Net-(A1-AGND) -> GND
- NMEA2000_CanController2 pad 3: Net-(Fuel_ADS1115-VDD) -> +3.3V
- PS1 pad 10_11: Net-(J4-GND) -> Net-(C5-Pad2)
- PS1 pad 12: Net-(J4-GND) -> Net-(C5-Pad2)
- PS1 pad 13: /GND_Page2 -> GND
- PS1 pad 18: Net-(J4-GND) -> Net-(C5-Pad2)
- PS1 pad 1_2: /5V_Page2 -> +5V
- PS1 pad 21: Net-(J4-GND) -> Net-(C5-Pad2)
- PS1 pad 25: /5V_Page2 -> +5V
- PS1 pad 6_7: /5V_Page2 -> +5V
- R11 pad 1: 3.3v_Page2 -> +3.3V
- R13 pad 1: 3.3v_Page2 -> +3.3V
- R15 pad 1: 3.3v_Page2 -> +3.3V
- R17 pad 2: Net-(Fuel_ADS1115-VDD) -> +3.3V
- R19 pad 2: Net-(J4-GND) -> GND
- R2 pad 1: 3.3v_Page2 -> +3.3V
- R20 pad 2: Net-(J4-GND) -> Net-(C5-Pad2)
- R21 pad 1: /5V_Page2 -> +5V
- R22 pad 1: /GND_Page2 -> GND
- R3 pad 1: 3.3v_Page2 -> +3.3V
- R5 pad 1: 3.3v_Page2 -> +3.3V
- R7 pad 1: 3.3v_Page2 -> +3.3V
- R9 pad 1: 3.3v_Page2 -> +3.3V
- U1 pad 1: Net-(J4-GND) -> GND
- U1 pad 10: Net-(J4-GND) -> GND
- U1 pad 11: /5V_Page2 -> unconnected-(U1-USB_VBUS-Pad11)
- U1 pad 14: Net-(J4-GND) -> GND
- U1 pad 2: Net-(J4-GND) -> GND
- U1 pad 37: Net-(J4-GND) -> GND
- U1 pad 40: Net-(J4-GND) -> GND
- U1 pad 41: Net-(J4-GND) -> GND
- U1 pad 43: Net-(J4-GND) -> GND
- U1 pad 5: Net-(J4-GND) -> GND
- U1 pad 57: Net-(J4-GND) -> GND
- U1 pad 58: Net-(J4-GND) -> GND
- U1 pad 60: Net-(J4-GND) -> GND
- U1 pad 61: Net-(J4-GND) -> GND
- U1 pad 64: Net-(J4-GND) -> GND
- U1 pad 65: Net-(J4-GND) -> GND
- U1 pad 77: Net-(J4-GND) -> GND
- U1 pad 78: Net-(J4-GND) -> GND
- U1 pad 80: Net-(J4-GND) -> GND
- U1 pad 81: Net-(J4-GND) -> GND
- U10 pad 1: Net-(J4-GND) -> GND
- U2 pad 3: Net-(Module1A-GND-Pad98) -> GND
- U3 pad 3: Net-(Module1A-GND-Pad98) -> GND
- U4 pad 3: Net-(Module1A-GND-Pad98) -> GND
- U5 pad 3: Net-(Module1A-GND-Pad98) -> GND
- U6 pad 3: Net-(Module1A-GND-Pad98) -> GND
- U7 pad 3: Net-(Module1A-GND-Pad98) -> GND
- U8 pad 3: Net-(Module1A-GND-Pad98) -> GND
- U9 pad 3: Net-(Module1A-GND-Pad98) -> GND
Routing:
- net GND: track 0.00 -> 554.2 mm, vias 0 -> 20
- net +3.3V: track 0.00 -> 526.6 mm, vias 0 -> 12
- net Net-(PS1-CTRL/UVLO): track 170.4 -> 636.0 mm
- net Net-(J4-GND): track 334.9 -> 0.00 mm
- net Net-(C5-Pad2): track 0.00 -> 334.9 mm
- net Net-(A1-GPIO21): track 0.00 -> 316.3 mm
- net 3.3v_Page2: track 293.0 -> 0.00 mm
- net Net-(Module1A-GPIO20): track 0.00 -> 252.2 mm, vias 0 -> 2
- net Net-(A1-GPIO22): track 0.00 -> 250.6 mm, vias 0 -> 2
- net Net-(Module1A-GPIO21): track 0.00 -> 247.2 mm, vias 0 -> 2
- net /5V_Page2: track 163.1 -> 0.00 mm
- net /GND_Page2: track 158.7 -> 0.00 mm
- net Net-(Module1A-GND-Pad98): track 135.2 -> 0.00 mm
- net Net-(J13-D2-): track 0.00 -> 127.3 mm
- net Net-(J13-D2+): track 0.00 -> 127.1 mm
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- added copper zone on B.Cu, net +3.3V
- added copper zone on In1.Cu, net +5V
- added copper zone on F.Cu, net GND
- added copper zone on In2.Cu, net GND
Other:
- board outline added: 394.5 x 186 mm
- copper layers 2 -> 6

Commit message: Updated from work
Parts:
- added C6: C1812W104KDRACTU, 100nFCapPretty:CAPC4532X185N, F.Cu at (253.9, 149.0)
- added M2: Fan_CPU_4pin, Connector:FanPinHeader_1x04_P2.54mm_Vertical, F.Cu at (327.4, 198.2)
- added REF**: MountingHole_4.3mm_M4, MountingHole:MountingHole_4.3mm_M4, F.Cu at (611.0, 150.0)
- added REF**: MountingHole_4.3mm_M4, MountingHole:MountingHole_4.3mm_M4, F.Cu at (464.5, 319.0)
- added REF**: MountingHole_4.3mm_M4, MountingHole:MountingHole_4.3mm_M4, F.Cu at (226.0, 319.0)
- added REF**: MountingHole_4.3mm_M4, MountingHole:MountingHole_4.3mm_M4, F.Cu at (428.5, 153.0)
- added REF**: MountingHole_4.3mm_M4, MountingHole:MountingHole_4.3mm_M4, F.Cu at (611.0, 319.0)
- added REF**: MountingHole_4.3mm_M4, MountingHole:MountingHole_4.3mm_M4, F.Cu at (226.0, 150.0)
- A1: value RaspberryPi_Pico_W -> RaspberryPi_Pico; footprint Module:RaspberryPi_Pico_W_SMD -> Module:RaspberryPi_Pico_SMD_HandSolder
- moved J14 5.60 mm to (251.4, 311.5)
- moved R20 2.99 mm to (259.0, 152.4)
- moved A1 0.11 mm to (296.3, 195.9)
Connections:
- J2 pad 1: unconnected-(J2-Pad1) -> Net-(J2-Pad1)
- Module1 pad 16: unconnected-(Module1A-FAN_TACHO-Pad16) -> Net-(M2-Tacho)
- Module1 pad 19: unconnected-(Module1A-FAN_PWM-Pad19) -> Net-(M2-PWM)
- R8 pad 1: unconnected-(R8-Pad1) -> Net-(R8-Pad1)
- R8 pad 2: unconnected-(R8-Pad2) -> Net-(J2-Pad1)
- U5 pad 1: unconnected-(U5-Pad1) -> Net-(R8-Pad1)
Routing:
- net +3.3V: track 526.6 -> 110.7 mm, vias 12 -> 15
- net GND: track 554.2 -> 508.4 mm, vias 20 -> 27
- net (no net): track 28.6 -> 0.00 mm
- net Net-(M2-Tacho): track 0.00 -> 21.6 mm
- net Net-(J2-Pad1): track 0.00 -> 21.3 mm
- net Net-(Module1A-GPIO22): track 112.9 -> 130.2 mm
- net Net-(PS1-SEQ): track 0.18 -> 16.6 mm
- net Net-(C5-Pad2): track 334.9 -> 350.3 mm
- net +5V: track 27.8 -> 38.2 mm, vias 4 -> 6
- net Net-(PS1-CTRL/UVLO): track 636.0 -> 646.3 mm
- net Net-(M2-PWM): track 0.00 -> 8.78 mm
- net Net-(R8-Pad1): track 0.00 -> 7.40 mm
- net Net-(A1-GPIO5): track 70.2 -> 63.9 mm
- net Net-(PS1-PG): track 7.64 -> 13.2 mm
- net Net-(A1-GPIO1): track 142.4 -> 145.5 mm
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- added copper zone on In2.Cu, net +5V
- added copper zone on In1.Cu, net GND
- removed copper zone on In1.Cu, net +5V
- removed copper zone on F.Cu, net GND
- removed copper zone on In2.Cu, net GND
Other:
- board size 394.5 x 186 mm -> 394.5 x 179 mm

Commit message: Fixed scheme
Parts:
- moved J6 6.50 mm to (434.2, 314.1)
- moved J13 3.02 mm to (380.2, 320.6)
- moved REF** 2.53 mm to (228.0, 151.6)
- moved J5 2.27 mm to (415.4, 314.1)
- moved REF** 1.83 mm to (609.5, 151.1)
- moved J3 0.05 mm to (407.2, 198.1)
Connections:
- Fuel_ADS1115 pad 8: unconnected-(Fuel_ADS1115-VDD-Pad8) -> +3.3V
- Module1 pad 65: unconnected-(Module1A-GND-Pad65) -> GND
- PS1 pad 10_11: Net-(C5-Pad2) -> GND
- PS1 pad 12: Net-(C5-Pad2) -> GND
- PS1 pad 13: GND -> Net-(PS1-VCC)
- PS1 pad 18: Net-(C5-Pad2) -> GND
- PS1 pad 21: Net-(C5-Pad2) -> GND
- R20 pad 2: Net-(C5-Pad2) -> GND
- R22 pad 1: GND -> Net-(PS1-VCC)
Routing:
- net Net-(C5-Pad2): track 350.3 -> 169.5 mm
- net +5V: track 38.2 -> 92.3 mm, vias 6 -> 5
- net GND: track 508.4 -> 456.1 mm
- net Net-(J13-SDA): track 119.4 -> 123.4 mm
- net Net-(L2-Pad1): track 14.3 -> 11.1 mm
- net Net-(PS1-VCC): track 0.00 -> 3.16 mm
- net Net-(J13-SCL): track 118.5 -> 121.4 mm
- net Net-(J13-HPD/HEAC-): track 119.4 -> 122.3 mm
- net Net-(J13-D2-): track 127.3 -> 130.2 mm
- net Net-(J13-D2+): track 127.8 -> 130.6 mm
- net Net-(J13-D1-): track 126.4 -> 129.3 mm
- net Net-(J13-D1+): track 126.1 -> 128.9 mm
- net Net-(J13-D0-): track 123.9 -> 126.7 mm
- net Net-(J13-D0+): track 124.5 -> 127.4 mm
- net Net-(J13-CK-): track 122.2 -> 125.0 mm
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
Commit message: Home push
Connections:
- A1 pad 33: GND -> unconnected-(A1-AGND-Pad33)
- A1 pad 36: +3.3V -> unconnected-(A1-3V3-Pad36)
- C1 pad 1: Net-(PS1-CTRL/UVLO) -> Net-(Module1A-GPIO20)
- C7 pad 1: Net-(PS1-CTRL/UVLO) -> Net-(Module1A-GPIO20)
- C8 pad 1: Net-(PS1-CTRL/UVLO) -> Net-(Module1A-GPIO20)
- Fuel_ADS1115 pad 3: Net-(Fuel_ADS1115-GND) -> GND
- J1 pad 4: Net-(Fuel_ADS1115-GND) -> GND
- J1 pad 5: Net-(PS1-CTRL/UVLO) -> Net-(Module1A-GPIO20)
- J14 pad 1: Net-(PS1-CTRL/UVLO) -> Net-(Module1A-GPIO20)
- J8 pad 1: Net-(Fuel_ADS1115-GND) -> GND
- Module1 pad 57: unconnected-(Module1A-SD_CLK-Pad57) -> Net-(J9-CLK)
- Module1 pad 61: unconnected-(Module1A-SD_DAT3-Pad61) -> Net-(J9-DAT3/CD)
- Module1 pad 62: unconnected-(Module1A-SD_CMD-Pad62) -> Net-(J9-CMD)
- Module1 pad 63: unconnected-(Module1A-SD_DAT0-Pad63) -> Net-(J9-DAT0)
- Module1 pad 67: unconnected-(Module1A-SD_DAT1-Pad67) -> Net-(J9-DAT1)
- Module1 pad 69: unconnected-(Module1A-SD_DAT2-Pad69) -> Net-(J9-DAT2)
- Module1 pad 86: +3.3V -> unconnected-(Module1A-+3.3v_(Output)-Pad86)
- PS1 pad 27: Net-(PS1-CTRL/UVLO) -> Net-(Module1A-GPIO20)
- PS1 pad 28: Net-(PS1-CTRL/UVLO) -> Net-(Module1A-GPIO20)
- PS1 pad 3: Net-(PS1-CTRL/UVLO) -> Net-(Module1A-GPIO20)
- PS1 pad 5: Net-(PS1-CTRL/UVLO) -> Net-(Module1A-GPIO20)
- PS1 pad 8: Net-(PS1-CTRL/UVLO) -> Net-(Module1A-GPIO20)
- PS1 pad 9: Net-(PS1-CTRL/UVLO) -> Net-(Module1A-GPIO20)
- U10 pad 3: Net-(PS1-CTRL/UVLO) -> Net-(Module1A-GPIO20)
- U10 pad 5: Net-(PS1-CTRL/UVLO) -> Net-(Module1A-GPIO20)
Routing:
- net Net-(PS1-CTRL/UVLO): track 647.2 -> 0.00 mm
- net Net-(Module1A-GPIO20): track 252.2 -> 899.4 mm
- net Net-(Fuel_ADS1115-GND): track 49.0 -> 0.00 mm
- net GND: track 456.1 -> 502.0 mm, vias 27 -> 26
- net unconnected-(A1-3V3-Pad36): track 0.00 -> 6.64 mm, vias 0 -> 1
- net +3.3V: track 113.0 -> 106.3 mm, vias 16 -> 15
- net unconnected-(A1-AGND-Pad33): track 0.00 -> 3.13 mm, vias 0 -> 1

Commit message: Work Changes and documentation
Parts:
- removed J6: USB3_A, StackedUSBPretty:MOLEX_484060003
- added C9: 10uf, Capacitor_SMD:C_0805_2012Metric, F.Cu at (433.1, 289.4)
- added F1: 3550-2, NewFuseHolderPretty:FUSE_3550-2, F.Cu at (258.5, 316.1)
- added J9: Micro_SD_Card_Det2, Connector_Card:SD_TE_2041021, F.Cu at (441.0, 310.1)
- added R23: 12k, Resistor_SMD:R_0805_2012Metric, F.Cu at (448.7, 289.5)
- added U11: RT9742BGJ5F, Package_TO_SOT_SMD:TSOT-23-5, F.Cu at (439.5, 289.6)
- J5: footprint StackedUSBPretty:MOLEX_484060003 -> CM5IO:MTCONN_UBAF30-D2011
- moved REF** 55.0 mm to (409.5, 318.1)
- moved J5 52.1 mm to (467.5, 314.2)
- moved J14 10.9 mm to (240.5, 311.5)
- moved J11 1.06 mm to (581.5, 312.1)
- moved J10 1.06 mm to (567.9, 312.1)
- moved J12 1.06 mm to (593.9, 312.1)
- moved J1 0.65 mm to (523.4, 309.6)
- moved J8 0.65 mm to (491.4, 309.6)
- moved J2 0.65 mm to (282.4, 295.5)
Connections:
- J14 pad 1: Net-(Module1A-GPIO20) -> Net-(F1-Pad1_1)
- Module1 pad 157: Net-(Module1B-USB3-1-RX_N) -> unconnected-(Module1B-USB3-1-RX_N-Pad157)
- Module1 pad 159: Net-(Module1B-USB3-1-RX_P) -> unconnected-(Module1B-USB3-1-RX_P-Pad159)
- Module1 pad 169: Net-(Module1B-USB3-1-TX_N) -> unconnected-(Module1B-USB3-1-TX_N-Pad169)
- Module1 pad 171: Net-(Module1B-USB3-1-TX_P) -> unconnected-(Module1B-USB3-1-TX_P-Pad171)
- Module1 pad 75: unconnected-(Module1A-SD_PWR_ON-Pad75) -> Net-(Module1A-SD_PWR_ON)
- Module1 pad 78: unconnected-(Module1A-GPIO_VREF(1.8v/3.3v_Input)-Pad78) -> +3.3V
- Module1 pad 86: unconnected-(Module1A-+3.3v_(Output)-Pad86) -> +3.3V
Routing:
- net Net-(Module1B-USB3-0-RX_N): track 0.00 -> 167.7 mm
- net Net-(Module1A-SD_PWR_ON): track 0.00 -> 163.8 mm, vias 0 -> 2
- net Net-(Module1B-USB3-0-RX_P): track 0.00 -> 158.0 mm
- net Net-(Module1B-USB3-0-D_P): track 0.00 -> 153.3 mm
- net Net-(Module1B-USB3-0-TX_P): track 0.00 -> 153.0 mm
- net Net-(Module1B-USB3-0-TX_N): track 0.00 -> 152.5 mm
- net Net-(Module1B-USB3-0-D_N): track 0.00 -> 151.9 mm
- net Net-(J9-DAT3/CD): track 0.00 -> 149.0 mm, vias 0 -> 2
- net Net-(J9-DAT2): track 0.00 -> 147.8 mm, vias 0 -> 2
- net Net-(J9-CLK): track 0.00 -> 141.9 mm, vias 0 -> 2
- net Net-(J9-DAT0): track 0.00 -> 136.4 mm, vias 0 -> 2
- net Net-(J9-CMD): track 0.00 -> 135.4 mm, vias 0 -> 2
- net Net-(J9-DAT1): track 0.00 -> 133.9 mm, vias 0 -> 2
- net Net-(Module1A-GPIO20): track 899.4 -> 936.6 mm
- net Net-(F1-Pad1_1): track 0.00 -> 24.9 mm
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
Commit message: fixed stuff at home
Parts:
- added C10: 10uf, Capacitor_SMD:C_0805_2012Metric, F.Cu at (391.9, 171.1)
- added C11: 10uf, Capacitor_SMD:C_0805_2012Metric, F.Cu at (396.0, 171.1)
- added C12: 100n, Capacitor_SMD:C_0805_2012Metric, F.Cu at (400.0, 171.1)
- added C13: 4.7nF, Capacitor_SMD:C_0805_2012Metric, F.Cu at (416.1, 170.0)
- added C14: 10uf, Capacitor_SMD:C_0805_2012Metric, F.Cu at (421.0, 170.9)
- added C15: 10uf, Capacitor_SMD:C_0805_2012Metric, F.Cu at (425.5, 170.9)
- added C16: 10uf, Capacitor_SMD:C_0805_2012Metric, F.Cu at (430.0, 170.9)
- added C17: 10uf, Capacitor_SMD:C_0805_2012Metric, F.Cu at (434.0, 170.9)
- added C18: 10uf, Capacitor_SMD:C_0805_2012Metric, F.Cu at (400.4, 176.5)
- added C19: 100n, Capacitor_SMD:C_0805_2012Metric, F.Cu at (356.6, 310.0)
- added C20: 100n, Capacitor_SMD:C_0805_2012Metric, F.Cu at (363.1, 316.0)
- added C21: 10uf, Capacitor_SMD:C_0805_2012Metric, F.Cu at (457.1, 293.5)
- added C22: 10uf, Capacitor_SMD:C_0805_2012Metric, F.Cu at (457.1, 289.5)
- added C23: 10uf, Capacitor_SMD:C_0805_2012Metric, F.Cu at (457.1, 285.5)
- added C24: 100uf, Capacitor_SMD:C_0805_2012Metric, F.Cu at (461.6, 287.5)
- added D1: LED, LED_SMD:LED_0805_2012Metric, F.Cu at (404.6, 211.5)
- added L3: 2.2uH, Inductor_SMD:L_0805_2012Metric, F.Cu at (411.6, 170.0)
- added R24: R, Resistor_SMD:R_0805_2012Metric, F.Cu at (408.9, 211.5)
- added R25: 100k, Resistor_SMD:R_0805_2012Metric, F.Cu at (410.1, 165.0)
- added R26: 100k 1%, Resistor_SMD:R_0805_2012Metric, F.Cu at (416.1, 174.0)
- added R27: 100k 1%, Resistor_SMD:R_0805_2012Metric, F.Cu at (416.1, 177.0)
- added R28: 15K 1%, Resistor_SMD:R_0805_2012Metric, F.Cu at (457.6, 302.4)
- added U12: AP3441SHE-7B, Package_DFN_QFN:DFN-8-1EP_2x2mm_P0.5mm_EP1.05x1.75mm, F.Cu at (406.0, 170.0)
- added U13: ASEK-32.768KHZ-L-R-T, Crystal:Crystal_SMD_3225-4Pin_3.2x2.5mm, F.Cu at (406.4, 176.8)
- added U14: RT9742SNGV, Package_TO_SOT_SMD:TSOT-23_HandSoldering, F.Cu at (363.8, 311.0)
- added U15: AP2553W6, Package_TO_SOT_SMD:SOT-23-6, F.Cu at (458.1, 297.1)
Connections:
- J13 pad 18: +5V -> Net-(J13-+5V)
- J3 pad 1: GND -> Net-(J3-GND-Pad1)
- J3 pad 10: unconnected-(J3-DAS/~{DSS}/~{LED1}-Pad10) -> Net-(J3-DAS/~{DSS}/~{LED1})
- J3 pad 12: +3.3V -> Net-(D1-A)
- J3 pad 14: +3.3V -> Net-(D1-A)
- J3 pad 15: GND -> Net-(J3-GND-Pad1)
- J3 pad 16: +3.3V -> Net-(D1-A)
- J3 pad 18: +3.3V -> Net-(D1-A)
- J3 pad 2: +3.3V -> Net-(D1-A)
- J3 pad 21: GND -> Net-(J3-GND-Pad1)
- J3 pad 27: GND -> Net-(J3-GND-Pad1)
- J3 pad 3: GND -> Net-(J3-GND-Pad1)
- J3 pad 33: GND -> Net-(J3-GND-Pad1)
- J3 pad 39: GND -> Net-(J3-GND-Pad1)
- J3 pad 4: +3.3V -> Net-(D1-A)
- J3 pad 45: GND -> Net-(J3-GND-Pad1)
- J3 pad 51: GND -> Net-(J3-GND-Pad1)
- J3 pad 57: GND -> Net-(J3-GND-Pad1)
- J3 pad 68: unconnected-(J3-SUSCLK-Pad68) -> Net-(J3-SUSCLK)
- J3 pad 70: +3.3V -> Net-(D1-A)
- J3 pad 71: GND -> Net-(J3-GND-Pad1)
- J3 pad 72: +3.3V -> Net-(D1-A)
- J3 pad 73: GND -> Net-(J3-GND-Pad1)
- J3 pad 74: +3.3V -> Net-(D1-A)
- J3 pad 75: GND -> Net-(J3-GND-Pad1)
- J3 pad 9: GND -> Net-(J3-GND-Pad1)
- J5 pad A1: +5V -> Net-(U15-OUT)
- J5 pad B1: +5V -> Net-(U15-OUT)
- Module1 pad 106: Net-(J3-~{PERST}) -> PCIE_PWR_EN
- Module1 pad 109: unconnected-(Module1B-PCIe_nRST-Pad109) -> Net-(J3-~{PERST})
- Module1 pad 163: /Sheet2/Sim7600_DP -> USB_DP
- Module1 pad 165: /Sheet2/Sim7600_DN -> USB_DN
- Module1 pad 191: GND -> Net-(J3-GND-Pad1)
- U1 pad 11: unconnected-(U1-USB_VBUS-Pad11) -> +5V
- U1 pad 12: /PI5_USB3_1_DN -> USB_DN
- U1 pad 13: /PI5_USB3_1_DP -> USB_DP
Routing:
- net Net-(J3-~{PERST}): track 30.6 -> 146.8 mm
- net Net-(D1-A): track 0.00 -> 99.9 mm, vias 0 -> 2
- net Net-(U15-OUT): track 0.00 -> 57.3 mm
- net PCIE_PWR_EN: track 0.00 -> 54.9 mm
- net GND: track 519.4 -> 565.9 mm, vias 30 -> 34
- net Net-(J3-GND-Pad1): track 0.00 -> 41.6 mm, vias 0 -> 3
- net Net-(U12-FB): track 0.00 -> 28.4 mm
- net +5V: track 97.5 -> 120.1 mm, vias 6 -> 8
- net Net-(J13-+5V): track 0.00 -> 22.5 mm
- net Net-(J3-SUSCLK): track 0.00 -> 16.9 mm
- net +3.3V: track 121.3 -> 111.0 mm, vias 17 -> 15
- net Net-(J3-DAS/~{DSS}/~{LED1}): track 0.00 -> 7.81 mm
- net Net-(A1-GPIO21): track 316.3 -> 321.7 mm
- net Net-(U12-LX): track 0.00 -> 3.70 mm
- net Net-(U15-ILIM): track 0.00 -> 3.42 mm
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