File: BoatPi.kicad_pcb (KiCad board)
At the start: 6 copper layers, 394.5 x 179 mm, 97 parts, among them J1 1432431, J10 CONSMA002-SMD-G, J11 CONSMA002-SMD-G, J12 CONSMA002-SMD-G, J13 HDMI_A_1.4, J14 Barrel_Jack_MountingPin, J2 1436987, J3 Bus_M.2_Socket_M, J4 JAE_SIM_Card_SF72S006, J5 USB3_A, J7 1436987, J8 1432431, J9 Micro_SD_Card_Det2, M2 Fan_CPU_4pin, U1 SIM7600E-H, U10 AP62301WU-7, U11 RT9742BGJ5F, U12 AP3441SHE-7B, U13 ASEK-32.768KHZ-L-R-T, U14 RT9742SNGV, U15 AP2553W6, U2 PC817, U3 PC817, U4 PC817, U5 PC817, U6 PC817, U7 PC817, U8 PC817, U9 PC817

Commit message: PCIE Changes
Parts:
- removed A1: RaspberryPi_Pico, Module:RaspberryPi_Pico_SMD_HandSolder
- added J6: 1436987, PHPretty:1436987, F.Cu at (306.0, 295.5)
- added K1: Relay_SPDT, Relay_THT:Relay_SPDT_Finder_36.11, F.Cu at (261.0, 294.8)
- added U16: SC0917, Pico2Pretty:MODULE_SC0917, F.Cu at (296.5, 196.1)
Connections:
- C1 pad 1: Net-(Module1A-GPIO20) -> Net-(PS1-CTRL/UVLO)
- C5 pad 2: Net-(C5-Pad2) -> GND
- C7 pad 1: Net-(Module1A-GPIO20) -> Net-(PS1-CTRL/UVLO)
- C7 pad 2: Net-(C5-Pad2) -> GND
- C8 pad 1: Net-(Module1A-GPIO20) -> Net-(PS1-CTRL/UVLO)
- C8 pad 2: Net-(C5-Pad2) -> GND
- F1 pad 2_1: Net-(Module1A-GPIO20) -> Net-(F1-Pad2_1)
- F1 pad 2_2: Net-(Module1A-GPIO20) -> Net-(F1-Pad2_1)
- J1 pad 5: Net-(Module1A-GPIO20) -> Net-(PS1-CTRL/UVLO)
- J14 pad 2: Net-(C5-Pad2) -> GND
- J3 pad 1: Net-(J3-GND-Pad1) -> GND
- J3 pad 15: Net-(J3-GND-Pad1) -> GND
- J3 pad 21: Net-(J3-GND-Pad1) -> GND
- J3 pad 27: Net-(J3-GND-Pad1) -> GND
- J3 pad 3: Net-(J3-GND-Pad1) -> GND
- J3 pad 33: Net-(J3-GND-Pad1) -> GND
- J3 pad 39: Net-(J3-GND-Pad1) -> GND
- J3 pad 41: Net-(J3-PETn0) -> /Sheet2/PET0_N
- J3 pad 43: Net-(J3-PETp0) -> /Sheet2/PET0_P
- J3 pad 45: Net-(J3-GND-Pad1) -> GND
- J3 pad 47: Net-(J3-PERn0) -> /Sheet2/PER0_N
- J3 pad 49: Net-(J3-PERp0) -> /Sheet2/PER0_P
- J3 pad 51: Net-(J3-GND-Pad1) -> GND
- J3 pad 57: Net-(J3-GND-Pad1) -> GND
- J3 pad 71: Net-(J3-GND-Pad1) -> GND
- J3 pad 73: Net-(J3-GND-Pad1) -> GND
- J3 pad 75: Net-(J3-GND-Pad1) -> GND
- J3 pad 9: Net-(J3-GND-Pad1) -> GND
- Module1 pad 1: unconnected-(Module1A-GND-Pad1) -> GND
- Module1 pad 107: unconnected-(Module1B-GND-Pad107) -> GND
- Module1 pad 111: unconnected-(Module1B-VBUS_EN-Pad111) -> VBUS_EN
- Module1 pad 113: unconnected-(Module1B-GND-Pad113) -> GND
- Module1 pad 114: unconnected-(Module1B-GND-Pad114) -> GND
- Module1 pad 116: Net-(J3-PERp0) -> /Sheet2/PET0_N
- Module1 pad 118: Net-(J3-PERn0) -> /Sheet2/PET0_P
- Module1 pad 119: unconnected-(Module1B-GND-Pad119) -> GND
- Module1 pad 120: unconnected-(Module1B-GND-Pad120) -> GND
- Module1 pad 122: Net-(J3-PETp0) -> /Sheet2/PER0_N
- Module1 pad 124: Net-(J3-PETn0) -> /Sheet2/PER0_P
- Module1 pad 125: unconnected-(Module1B-GND-Pad125) -> GND
- Module1 pad 126: unconnected-(Module1B-GND-Pad126) -> GND
- Module1 pad 13: unconnected-(Module1A-GND-Pad13) -> GND
- Module1 pad 131: unconnected-(Module1B-GND-Pad131) -> GND
- Module1 pad 132: unconnected-(Module1B-GND-Pad132) -> GND
- Module1 pad 137: unconnected-(Module1B-GND-Pad137) -> GND
- Module1 pad 138: unconnected-(Module1B-GND-Pad138) -> GND
- Module1 pad 14: unconnected-(Module1A-GND-Pad14) -> GND
- Module1 pad 144: unconnected-(Module1B-GND-Pad144) -> GND
- Module1 pad 150: unconnected-(Module1B-GND-Pad150) -> GND
- Module1 pad 155: unconnected-(Module1B-GND-Pad155) -> GND
- Module1 pad 156: unconnected-(Module1B-GND-Pad156) -> GND
- Module1 pad 161: unconnected-(Module1B-GND-Pad161) -> GND
- Module1 pad 162: unconnected-(Module1B-GND-Pad162) -> GND
- Module1 pad 167: unconnected-(Module1B-GND-Pad167) -> GND
- Module1 pad 168: unconnected-(Module1B-GND-Pad168) -> GND
- Module1 pad 173: unconnected-(Module1B-GND-Pad173) -> GND
- Module1 pad 174: unconnected-(Module1B-GND-Pad174) -> GND
- Module1 pad 179: unconnected-(Module1B-GND-Pad179) -> GND
- Module1 pad 180: unconnected-(Module1B-GND-Pad180) -> GND
- Module1 pad 185: unconnected-(Module1B-GND-Pad185) -> GND
- Module1 pad 186: unconnected-(Module1B-GND-Pad186) -> GND
- Module1 pad 191: Net-(J3-GND-Pad1) -> GND
- Module1 pad 197: unconnected-(Module1B-GND-Pad197) -> GND
- Module1 pad 198: unconnected-(Module1B-GND-Pad198) -> GND
- Module1 pad 2: unconnected-(Module1A-GND-Pad2) -> GND
- Module1 pad 22: unconnected-(Module1A-GND-Pad22) -> GND
- Module1 pad 23: unconnected-(Module1A-GND-Pad23) -> GND
- Module1 pad 32: unconnected-(Module1A-GND-Pad32) -> GND
- Module1 pad 33: unconnected-(Module1A-GND-Pad33) -> GND
- Module1 pad 39: unconnected-(Module1A-GPIO8-Pad39) -> GPIO8
- Module1 pad 41: unconnected-(Module1A-GPIO25-Pad41) -> GPIO25
- Module1 pad 42: unconnected-(Module1A-GND-Pad42) -> GND
- Module1 pad 45: unconnected-(Module1A-GPIO24-Pad45) -> GPIO24
- Module1 pad 52: unconnected-(Module1A-GND-Pad52) -> GND
- Module1 pad 53: unconnected-(Module1A-GND-Pad53) -> GND
- Module1 pad 59: unconnected-(Module1A-GND-Pad59) -> GND
- Module1 pad 60: unconnected-(Module1A-GND-Pad60) -> GND
- Module1 pad 66: unconnected-(Module1A-GND-Pad66) -> GND
- Module1 pad 7: unconnected-(Module1A-GND-Pad7) -> GND
- Module1 pad 71: unconnected-(Module1A-GND-Pad71) -> GND
- Module1 pad 74: unconnected-(Module1A-GND-Pad74) -> GND
- Module1 pad 8: unconnected-(Module1A-GND-Pad8) -> GND
- PS1 pad 27: Net-(Module1A-GPIO20) -> Net-(PS1-CTRL/UVLO)
- PS1 pad 28: Net-(Module1A-GPIO20) -> Net-(PS1-CTRL/UVLO)
- PS1 pad 3: Net-(Module1A-GPIO20) -> Net-(PS1-CTRL/UVLO)
- PS1 pad 5: Net-(Module1A-GPIO20) -> Net-(PS1-CTRL/UVLO)
- PS1 pad 8: Net-(Module1A-GPIO20) -> Net-(PS1-CTRL/UVLO)
- PS1 pad 9: Net-(Module1A-GPIO20) -> Net-(PS1-CTRL/UVLO)
- U10 pad 3: Net-(Module1A-GPIO20) -> Net-(PS1-CTRL/UVLO)
- U10 pad 5: Net-(Module1A-GPIO20) -> Net-(PS1-CTRL/UVLO)
- U13 pad 2: unconnected-(U13-GND-Pad2) -> GND
Routing:
- net Net-(Module1A-GPIO20): track 936.6 -> 246.0 mm
- net Net-(PS1-CTRL/UVLO): track 0.00 -> 635.7 mm
- net GND: track 565.9 -> 971.2 mm, vias 34 -> 51
- net USB_DP: track 0.00 -> 215.3 mm, vias 0 -> 2
- net USB_DN: track 0.00 -> 212.2 mm, vias 0 -> 2
- net Net-(C5-Pad2): track 165.7 -> 0.00 mm
- net VBUS_EN: track 0.00 -> 137.7 mm, vias 0 -> 2
- net GPIO8: track 0.00 -> 116.6 mm, vias 0 -> 1
- net GPIO24: track 0.00 -> 115.6 mm, vias 0 -> 1
- net GPIO25: track 0.00 -> 114.5 mm, vias 0 -> 1
- net Net-(F1-Pad2_1): track 0.00 -> 77.2 mm
- net Net-(J6-Pad2): track 0.00 -> 47.0 mm
- net Net-(J3-GND-Pad1): track 41.6 -> 0.00 mm, vias 3 -> 0
- net PCIE_PWR_EN: track 54.9 -> 92.2 mm
- net Net-(D1-A): track 99.9 -> 129.7 mm
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
Commit message: diff pairs
Connections:
- net Net-(NMEA2000_CanController2-CANL) renamed /CAN+
- J1 pad 1: unconnected-(J1-Pad1) -> GND
- J1 pad 2: Net-(NMEA2000_CanController2-STBY) -> /CAN-
- J1 pad 4: GND -> Net-(PS1-CTRL/UVLO)
- J1 pad 5: Net-(PS1-CTRL/UVLO) -> GND
- J1 pad MH1: unconnected-(J1-PadMH1) -> GND
- NMEA2000_CanController2 pad 7: unconnected-(NMEA2000_CanController2-CANH-Pad7) -> /CAN-
- NMEA2000_CanController2 pad 8: Net-(NMEA2000_CanController2-STBY) -> GND
Routing:
- net /Sheet2/PER0_P: track 0.00 -> 35.0 mm, vias 0 -> 2
- net /Sheet2/PER0_N: track 0.00 -> 28.9 mm, vias 0 -> 2
- net /CAN-: track 0.00 -> 15.2 mm
- net Net-(NMEA2000_CanController2-STBY): track 10.4 -> 0.00 mm
- net /Sheet2/PET0_P: track 23.1 -> 27.3 mm
- net /Sheet2/PET0_N: track 24.3 -> 25.3 mm
- net /CAN+: track 14.4 -> 15.4 mm
