File: BoatPi.kicad_pcb (KiCad board)
At the start: 6 copper layers, 394.5 x 179 mm, 99 parts, among them J1 1432431, J10 CONSMA002-SMD-G, J11 CONSMA002-SMD-G, J12 CONSMA002-SMD-G, J13 HDMI_A_1.4, J14 Barrel_Jack_MountingPin, J2 1436987, J3 Bus_M.2_Socket_M, J4 JAE_SIM_Card_SF72S006, J5 USB3_A, J6 1436987, J7 1436987, J8 1432431, J9 Micro_SD_Card_Det2, K1 Relay_SPDT, M2 Fan_CPU_4pin, U1 SIM7600E-H, U10 AP62301WU-7, U11 RT9742BGJ5F, U12 AP3441SHE-7B, U13 ASEK-32.768KHZ-L-R-T, U14 RT9742SNGV, U15 AP2553W6, U16 SC0917, U2 PC817, U3 PC817, U4 PC817, U5 PC817, U6 PC817, U7 PC817, U8 PC817, U9 PC817

Commit message: Fixes from datasheets
Parts:
- J13: footprint Connector_Video:HDMI_A_Amphenol_10029449-x01xLF_Horizontal -> CM5IO:EDAC 690-019-298-412
- J9: footprint Connector_Card:SD_TE_2041021 -> CM5IO:SDCARD_MOLEX_503398-1892
- U12: footprint Package_DFN_QFN:DFN-8-1EP_2x2mm_P0.5mm_EP1.05x1.75mm -> Package_DFN_QFN:DFN-8-1EP_3x3mm_P0.65mm_EP1.7x2.05mm
- U13: footprint Crystal:Crystal_SMD_3225-4Pin_3.2x2.5mm -> Crystal:Crystal_SMD_3225-4Pin_3.2x2.5mm_HandSoldering
- U15: footprint Package_TO_SOT_SMD:SOT-23-6 -> Package_TO_SOT_SMD:SOT-23-6_Handsoldering
- moved J13 7.07 mm to (380.5, 313.6)
- moved J9 6.51 mm to (438.8, 316.2)
- moved J4 2.15 mm to (547.5, 314.4)
- moved U1 0.08 mm to (578.0, 268.9)
Connections:
- net Net-(J13-CK+) renamed /Sheet2/HDMI_CK+
- net Net-(J13-CK-) renamed /Sheet2/HDMI_CK-
- net Net-(J13-D0+) renamed /Sheet2/HDMI_DO+
- net Net-(J13-D0-) renamed /Sheet2/HDMI_DO-
- net Net-(J13-D1+) renamed /Sheet2/HDMI_D1+
- net Net-(J13-D1-) renamed /Sheet2/HDMI_D1-
- net Net-(J13-D2+) renamed /Sheet2/HDMI_D2+
- net Net-(J13-D2-) renamed /Sheet2/HDMI_D2-
- net Net-(Module1B-USB3-0-D_N) renamed /Sheet2/USB_D-
- net Net-(Module1B-USB3-0-D_P) renamed /Sheet2/USB_D+
- net Net-(Module1B-USB3-0-RX_N) renamed /Sheet2/USB_SSRX+
- net Net-(Module1B-USB3-0-RX_P) renamed /Sheet2/USB_SSRX-
- net Net-(Module1B-USB3-0-TX_N) renamed /Sheet2/USB+SSTX-
- net Net-(Module1B-USB3-0-TX_P) renamed /Sheet2/USB_SSTX+
- Fuel_ADS1115 pad 10: unconnected-(Fuel_ADS1115-SCL-Pad10) -> GPIO3
- Fuel_ADS1115 pad 9: unconnected-(Fuel_ADS1115-SDA-Pad9) -> GPIO2
- J4 pad CSW: unconnected-(J4-PadCSW) -> Net-(U1-USIM_DET)
- J4 pad DSW: unconnected-(J4-PadDSW) -> Net-(U1-USIM_DET)
- J4 pad SH: unconnected-(J4-PadSH)_9 -> GND
- Module1 pad 56: unconnected-(Module1A-GPIO3-Pad56) -> GPIO3
- Module1 pad 58: unconnected-(Module1A-GPIO2-Pad58) -> GPIO2
- U1 pad 53: unconnected-(U1-USIM_DET-Pad53) -> Net-(U1-USIM_DET)
Routing:
- net GPIO3: track 0.00 -> 315.5 mm, vias 0 -> 2
- net GPIO2: track 0.00 -> 232.3 mm, vias 0 -> 2
- net Net-(U1-USIM_DET): track 0.00 -> 101.6 mm
- net GND: track 971.2 -> 1025.8 mm, vias 51 -> 67
- net Net-(J9-VDD): track 16.0 -> 57.2 mm
- net Net-(J9-DAT1): track 133.9 -> 158.2 mm
- net /Sheet2/USB_SSRX-: track 158.0 -> 180.5 mm
- net Net-(J9-DAT0): track 136.4 -> 156.9 mm
- net Net-(Module1A-SD_PWR_ON): track 163.8 -> 148.7 mm
- net Net-(J9-CLK): track 141.9 -> 155.7 mm
- net Net-(J9-CMD): track 135.4 -> 147.6 mm
- net Net-(Module1A-GPIO27): track 159.4 -> 168.8 mm
- net Net-(J4-RST): track 41.2 -> 46.4 mm
- net Net-(J4-VPP/SWP): track 46.1 -> 51.1 mm
- net Net-(J9-DAT3/CD): track 149.0 -> 153.3 mm
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
Commit message: Final Updates
Parts:
- removed C3, C4: EEEFN1C220R, 22uFCap:CAP_EEEFN1C220R
- removed L1: L, Inductor_SMD:L_0805_2012Metric
- added C25: 100nF, Capacitor_SMD:C_0805_2012Metric, F.Cu at (556.0, 291.0)
- added C26: 22pF_NM, Capacitor_SMD:C_0805_2012Metric, F.Cu at (562.5, 294.5)
- added C27: 22pF_NM, Capacitor_SMD:C_0805_2012Metric, F.Cu at (552.0, 281.5)
- added C28: 22pF_NM, Capacitor_SMD:C_0805_2012Metric, F.Cu at (563.5, 288.0)
- added C29: 100nF, Capacitor_SMD:C_0805_2012Metric, F.Cu at (539.0, 240.0)
- added D2: ESDA6V1W5, TVSPretty:SOT65P210X110-5N, F.Cu at (552.6, 302.9)
- added D3: TVS-bidirectional Diode, Diode_SMD:D_0805_2012Metric, F.Cu at (539.1, 236.0)
- added F2: 2A, Fuse:Fuse_0805_2012Metric, F.Cu at (582.5, 239.8)
- added Q2: BC107, Package_TO_SOT_THT:TO-18-3, F.Cu at (543.5, 248.2)
- added R29: 22 Ohm, Resistor_SMD:R_0805_2012Metric, F.Cu at (556.5, 312.5)
- added R30: 22 Ohm, Resistor_SMD:R_0805_2012Metric, F.Cu at (542.5, 296.4)
- added R31: 22 Ohm, Resistor_SMD:R_0805_2012Metric, F.Cu at (547.4, 299.1)
- added R32: 0 Ohm, Resistor_SMD:R_0805_2012Metric, F.Cu at (559.0, 259.9)
- added R33: 4.7K, Resistor_SMD:R_0805_2012Metric, F.Cu at (544.1, 262.5)
- added R34: 47k, Resistor_SMD:R_0805_2012Metric, F.Cu at (538.0, 245.9)
- added R35: 470R, Resistor_SMD:R_0805_2012Metric, F.Cu at (587.6, 235.0)
- C1: value EEEFN1J100L -> C_Polarized_Small_US; footprint 10uFCapPretty:CAP_EEEFN1J100L -> Capacitor_SMD:C_0805_2012Metric
- R18, R19: value R -> 470R
- U10: value AP62301WU-7 -> MIC29302AWU; footprint APBuckPretty:SOT95P280X100-6N -> Package_TO_SOT_SMD:TO-263-5_TabPin3
- moved C1 32.1 mm to (587.5, 249.5)
- moved C2 14.7 mm to (588.9, 244.5)
- moved U10 14.5 mm to (585.2, 220.9), turned to 90 degrees
- moved R18 6.92 mm to (587.6, 240.0), turned to 0 degrees
- moved R19 3.14 mm to (594.1, 235.0), turned to 0 degrees
Connections:
- C1 pad 1: Net-(PS1-CTRL/UVLO) -> Net-(U10-VOUT)
- C2 pad 1: Net-(U10-BST) -> Net-(U10-VOUT)
- C2 pad 2: Net-(U10-SW) -> GND
- J4 pad C6: Net-(J4-VPP/SWP) -> unconnected-(J4-VPP/SWP-PadC6)
- J4 pad C7: unconnected-(J4-I/O-PadC7) -> Net-(J4-I/O)
- Module1 pad 25: Net-(Module1A-GPIO21) -> unconnected-(Module1A-GPIO21-Pad25)
- NMEA2000_CanController2 pad 3: +3.3V -> +5V
- R18 pad 1: Net-(C3-Pad1) -> Net-(U10-VOUT)
- R18 pad 2: Net-(U10-FB) -> GND
- R19 pad 1: Net-(U10-FB) -> Net-(U10-ADJ)
- U1 pad 17: Net-(J4-VPP/SWP) -> Net-(U1-USIM_DATA)
- U1 pad 18: Net-(J4-RST) -> Net-(U1-USIM_RST)
- U1 pad 19: Net-(J4-CLK) -> Net-(U1-USIM_CLK)
- U1 pad 3: Net-(Module1A-GPIO21) -> Net-(U1-PWRKEY)
- U1 pad 38: Net-(C3-Pad1) -> Net-(U10-VOUT)
- U1 pad 39: Net-(C3-Pad1) -> Net-(U10-VOUT)
- U1 pad 4: Net-(Module1A-GPIO20) -> Net-(D3-A)
- U1 pad 62: Net-(C3-Pad1) -> Net-(U10-VOUT)
- U1 pad 63: Net-(C3-Pad1) -> Net-(U10-VOUT)
- U10 pad 1: GND -> Net-(U10-EN)
- U10 pad 2: Net-(U10-SW) -> Net-(U10-EN)
- U10 pad 3: Net-(PS1-CTRL/UVLO) -> GND
- U10 pad 4: Net-(U10-FB) -> Net-(U10-VOUT)
- U10 pad 5: Net-(PS1-CTRL/UVLO) -> Net-(U10-ADJ)
Routing:
- net Net-(Module1A-GPIO21): track 247.4 -> 0.00 mm, vias 2 -> 0
- net Net-(C3-Pad1): track 122.8 -> 0.00 mm
- net Net-(U10-VOUT): track 0.00 -> 87.0 mm
- net Net-(PS1-CTRL/UVLO): track 636.8 -> 566.4 mm
- net Net-(D3-A): track 0.00 -> 61.1 mm
- net Net-(J4-VPP/SWP): track 51.1 -> 0.00 mm
- net Net-(U1-USIM_DATA): track 0.00 -> 44.6 mm
- net Net-(U1-USIM_RST): track 0.00 -> 37.2 mm
- net Net-(U1-USIM_CLK): track 0.00 -> 31.3 mm
- net Net-(J4-RST): track 46.4 -> 16.5 mm
- net Net-(U10-SW): track 25.0 -> 0.00 mm
- net Net-(J4-I/O): track 0.00 -> 24.6 mm
- net Net-(U10-FB): track 21.0 -> 0.00 mm
- net Net-(Q2-B): track 0.00 -> 20.9 mm
- net Net-(Module1A-GPIO20): track 246.0 -> 226.3 mm
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
Commit message: Label Fixes
Parts:
- moved REF** 7.00 mm to (602.5, 151.0)
- moved REF** 7.00 mm to (604.0, 318.9)
Routing:
- net Net-(Q2-B): track 20.9 -> 21.6 mm
Other:
- board size 394.5 x 179 mm -> 388.5 x 179 mm
Changed lines of the file:
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@@
 		(tags "capacitor")
 		(property "Reference" "C22"
-			(at 4.05 -0.735 0)
+			(at 3.55 0 0)
 			(layer "F.SilkS")
 			(effects
@@
 		)
 		(property "Value" "100nF"
-			(at 0 1.68 0)
+			(at 5.95 0 0)
 			(layer "F.Fab")
 			(effects
@@
 		(tags "capacitor")
 		(property "Reference" "C14"
-			(at 0 -1.68 90)
+			(at -3.45 0 90)
 			(layer "F.SilkS")
 			(effects
@@
 		)
 		(property "Value" "HDMI_A_1.4"
-			(at -6.1 -2.9 0)
+			(at 0.05 6.4125 0)
 			(layer "F.SilkS")
 			(effects
@@
 	(footprint "MountingHole:MountingHole_4.3mm_M4"
 		(layer "F.Cu")
-		(at 609.5 151.05)
+		(at 602.5 151)
 		(descr "Mounting Hole 4.3mm, no annular, M4")
 		(tags "mounting hole 4.3mm no annular m4")
@@
 		(tags "resistor")
 		(property "Reference" "R17"
-			(at 0 -1.65 90)
+			(at -0.6875 -2.0075 90)
 			(layer "F.SilkS")
 			(effects
@@
 		)
 		(property "Value" "270Ohm"
-			(at 0 1.65 90)
+			(at 2.3125 1.65 90)
 			(layer "F.Fab")
 			(effects
@@
 		)
 		(property "Value" "CONSMA002-SMD-G"
-			(at 7.3 13.585 0)
+			(at -0.42 7.86 0)
 			(layer "F.Fab")
 			(effects
@@
 		(tags "capacitor")
 		(property "Reference" "C9"
-			(at 0 -1.68 90)
+			(at -2.45 0.15 0)
 			(layer "F.SilkS")
 			(effects
@@
 		(tags "resistor")
 		(property "Reference" "R27"
-			(at 0 -1.65 0)
+			(at -1.4125 -1.65 0)
 			(layer "F.SilkS")
 			(effects
@@
 		)
 		(property "Value" "100k 1%"
-			(at 0 1.65 0)
+			(at -5.4125 0 0)
 			(layer "F.Fab")
 			(effects
@@
 		)
 		(property "Value" "MountingHole_4.3mm_M4"
-			(at 0 5.3 0)
+			(at 5.5 3.5 0)
 			(layer "F.Fab")
 			(effects
@@
 		(at 493.77 283.9)
 		(property "Reference" "Fuel_ADS1115"
-			(at 0.175 -2.635 0)
+			(at 1.23 -2.635 0)
 			(layer "F.SilkS")
 			(effects
@@
 		)
 		(property "Value" "ADS1115BQDGSRQ1"
-			(at 7.795 2.635 0)
+			(at 6.73 2.6 0)
 			(layer "F.Fab")
 			(effects
@@
 		(tags "capacitor")
 		(property "Reference" "C13"
-			(at 0 -1.68 0)
+			(at 0.95 -2 0)
 			(layer "F.SilkS")
 			(effects
@@
 		(tags "Raspberry Pi 5 Compute Module")
 		(property "Reference" "Module1"
-			(at 18.38 -5.08 270)
+			(at 16.04 -41.9 180)
 			(layer "F.SilkS")
 			(effects
@@
 		)
 		(property "Value" "ComputeModule5-CM5"
-			(at 16.52 0.19 0)
+			(at 16.5 -46.4 0)
 			(layer "F.Fab")
 			(effects
@@
 		(tags "capacitor")
 		(property "Reference" "C15"
-			(at 0 -1.68 90)
+			(at -2.95 0 90)
 			(layer "F.SilkS")
 			(effects
@@
 		)
 		(property "Value" "Barrel_Jack_MountingPin"
-			(at 0 13 0)
+			(at 0 -5.5 0)
 			(layer "F.Fab")
 			(effects
@@
 	(footprint "MountingHole:MountingHole_4.3mm_M4"
 		(layer "F.Cu")
-		(at 611 319)
+		(at 604 318.95)
 		(descr "Mounting Hole 4.3mm, no annular, M4")
 		(tags "mounting hole 4.3mm no annular m4")
@@
 		)
 		(property "Value" "MountingHole_4.3mm_M4"
-			(at 0 5.3 0)
+			(at -4 4.05 0)
 			(layer "F.Fab")
 			(effects
@@
 		)
 		(property "Value" "RT9742BGJ5F"
-			(at 0 2.4 0)
+			(at 2.4875 2.45 0)
 			(layer "F.Fab")
 			(effects
@@
 		)
 		(property "Value" "10uf"
-			(at 0 1.68 0)
+			(at 3.95 0 0)
 			(layer "F.Fab")
 			(effects
@@
 		(tags "resistor")
 		(property "Reference" "R34"
-			(at 0 -1.65 90)
+			(at 1.0875 -2 90)
 			(layer "F.SilkS")
 			(effects
@@
 		(tags "DFN NoLead")
 		(property "Reference" "U12"
-			(at 0 -2.45 0)
+			(at 0 -3 0)
 			(layer "F.SilkS")
 			(effects
@@
 		(tags "resistor")
 		(property "Reference" "R18"
-			(at 0 -1.65 0)
+			(at 0.9125 -1.65 0)
 			(layer "F.SilkS")
 			(effects
@@
 		)
 		(property "Value" "Micro_SD_Card_Det2"
-			(at 3.719055 8.349145 0)
+			(at -14.78 -0.175 0)
 			(layer "F.Fab")
 			(effects
@@
 		)
 		(property "Value" "CONSMA002-SMD-G"
-			(at 7.3 13.585 0)
+			(at 0.08 7.95 0)
 			(layer "F.Fab")
 			(effects
@@
 		(tags "capacitor")
 		(property "Reference" "C10"
-			(at 0 -1.68 90)
+			(at -3.05 -0.05 90)
 			(layer "F.SilkS")
 			(effects
@@
 		(tags "capacitor")
 		(property "Reference" "C21"
-			(at 4.05 -0.05 0)
+			(at 3.55 0 0)
 			(layer "F.SilkS")
 			(effects
@@
 		(tags "resistor")
 		(property "Reference" "R28"
-			(at 0 -1.65 90)
+			(at 0.0875 -1.9125 90)
 			(layer "F.SilkS")
 			(effects
@@
 		(tags "resistor")
 		(property "Reference" "R23"
-			(at 0 -1.65 90)
+			(at -2.5 0.2375 0)
 			(layer "F.SilkS")
 			(effects
@@
 		(tags "capacitor")
 		(property "Reference" "C17"
-			(at 0 -1.68 90)
+			(at -2.95 0.5 90)
 			(layer "F.SilkS")
 			(effects
@@
 		)
 		(property "Value" "C_Polarized_Small_US"
-			(at 0 1.68 0)
+			(at 10.95 1 0)
 			(layer "F.Fab")
 			(effects
@@
 		(at 407.225 198.05 90)
 		(property "Reference" "J3"
-			(at -7.62 -10.287 90)
+			(at -5.95 -7.225 90)
 			(layer "F.SilkS")
 			(effects
@@
 		)
 		(property "Value" "Fan_CPU_4pin"
-			(at 4.05 4.35 0)
+			(at 0.58 4.84 0)
 			(layer "F.Fab")
 			(effects
@@
 		(tags "resistor")
 		(property "Reference" "R26"
-			(at 0 -1.65 0)
+			(at -3.0875 0 0)
 			(layer "F.SilkS")
 			(effects
@@
 		)
 		(property "Value" "100k 1%"
-			(at 0 1.65 0)
+			(at 5.4125 0 0)
 			(layer "F.Fab")
 			(effects
@@
 		)
 		(property "Value" "3550-2"
-			(at -3.415 8.135 0)
+			(at 0 0 0)
 			(layer "F.Fab")
 			(effects
@@
 		)
 		(property "Value" "C1812W104KDRACTU"
-			(at 0.24 2.35 0)
+			(at 7.057 0 0)
 			(layer "F.Fab")
 			(effects
@@
 		(tags "capacitor")
 		(property "Reference" "C23"
-			(at 4.55 -0.05 0)
+			(at 3.55 -0.05 0)
 			(layer "F.SilkS")
 			(effects
@@
 		(tags "resistor")
 		(property "Reference" "R35"
-			(at 3 -0.44 0)
+			(at 2.4125 -1.5 0)
 			(layer "F.SilkS")
 			(effects
@@
 		)
 		(property "Value" "CONSMA002-SMD-G"
-			(at 7.3 13.585 0)
+			(at 0 9.36 0)
 			(layer "F.Fab")
 			(effects
@@
 		(tags "MCP2562FD-H/SN ")
 		(property "Reference" "NMEA2000_CanController2"
-			(at 0 -5.985 270)
+			(at -1.0378 -4.985 270)
 			(unlocked yes)
 			(layer "F.SilkS")
@@
 		)
 		(property "Value" "MCP2562FD-H/SN"
-			(at 0 -8.985 270)
+			(at 0 -6.985 270)
 			(unlocked yes)
 			(layer "F.Fab")
@@
 		)
 		(fp_text user "*"
-			(at 0.9622 -3.985 270)
+			(at -0.0378 -0.985 270)
 			(unlocked yes)
 			(layer "F.SilkS")
@@
 		)
 		(fp_text user "*"
-			(at -2.0378 -4.485 90)
+			(at 0 0 90)
 			(layer "F.SilkS")
 			(effects
@@
 		(tags "capacitor")
 		(property "Reference" "C11"
-			(at 0 -1.68 90)
+			(at -3.05 0 90)
 			(layer "F.SilkS")
 			(effects
@@
 		(tags "USB3 TypeA")
 		(property "Reference" "J5"
-			(at 0 -0.5 0)
+			(at 0 2.34 0)
 			(unlocked yes)
 			(layer "F.SilkS")
@@
 		)
 		(property "Value" "USB3_A"
-			(at 0 1 0)
+			(at 0 3.84 0)
 			(unlocked yes)
 			(layer "F.Fab")
@@
 		)
 		(fp_text user "${REFERENCE}"
-			(at 0 2.5 0)
+			(at 0 5.34 0)
 			(unlocked yes)
 			(layer "F.Fab")
@@
 		(tags "capacitor")
 		(property "Reference" "C12"
-			(at 0 -1.68 90)
+			(at -3.55 0 90)
 			(layer "F.SilkS")
 			(effects
@@
 		)
 		(property "Value" "100n"
-			(at 0 1.68 90)
+			(at -0.05 1.68 90)
 			(layer "F.Fab")
 			(effects
@@
 		(tags "SOT-23-6 Handsoldering")
 		(property "Reference" "U15"
-			(at 0 -2.9 270)
+			(at 0 -3.95 270)
 			(layer "F.SilkS")
 			(effects
@@
 		)
 		(property "Value" "AP2553W6"
-			(at 0 2.9 270)
+			(at 1.8625 4.55 270)
 			(layer "F.Fab")
 			(effects
@@
 		(tags "capacitor")
 		(property "Reference" "C16"
-			(at 0 -1.68 90)
+			(at -2.95 0 90)
 			(layer "F.SilkS")
 			(effects
@@
 	(gr_rect
 		(start 221.25 145)
-		(end 615.75 324)
+		(end 609.75 324)
 		(stroke
 			(width 0.05)
@@
 	(segment
 		(start 544.721961 249.491961)
-		(end 540.666961 249.491961)
+		(end 539.491961 249.491961)
 		(width 0.2)
 		(layer "F.Cu")
@@
 	)
 	(segment
-		(start 540.666961 249.491961)
-		(end 538 246.825)
+		(start 539.491961 249.491961)
+		(end 538 248)
 		(width 0.2)
 		(layer "F.Cu")
@@
 		(width 0.2)
 		(layer "F.Cu")
+		(net 364)
+	)
+	(segment
+		(start 538 248)
+		(end 538 246.825)
+		(width 0.2)
+		(layer "F.Cu")
